File: hardware/2kwMotorController.kicad_pcb (KiCad board)
At the start: 4 copper layers, 170.2 x 81.3 mm, 147 parts, among them Q1 DMG4712SSS, Q2 DMG4712SSS, Q3 IRFP4468, Q4 IRFP4468, Q5 IRFP4468, Q6 IRFP4468, Q7 IRFP4468, Q8 IRFP4468, Q9 DMT10H010LK3, U1 LM358, U10 LF33ABDT, U11 TM4C1294KCPDT, U12 Si8640, U13 MIC4127, U14 LM5102, U15 LM5102, U16 MCP1501T-30E, U17 MIC5225-5.0, U18 SN65HVD231D, U19 MIC4127, U2 MCP6001, U20 Si8640, U3 LAH-100P, U4 LOC110, U5 MCP6001, U6 ADA4805-1, U7 LT3471, U9 MIC5225-5.0, Y1 NX5032GA

Commit message: Added most footprints, did non-power layout
Parts:
- added C62: 2.2u, Capacitors_SMD:C_0603, F.Cu at (287.8, 10.0)
- added C63: 2.2u, Capacitors_SMD:C_0603, F.Cu at (301.2, 10.0)
- added C64: 100n, Capacitors_SMD:C_0603, F.Cu at (306.8, 10.0)
- added C65: 100n, Capacitors_SMD:C_0603, F.Cu at (269.8, 14.4)
- added P1: CONN_01X02_CBAT, 2kwMotorController:TERM_2P_2-5_1990009, F.Cu at (159.8, 99.4)
- added P2: CONN_02X05_JTAG, Pin_Headers:Pin_Header_Straight_2x05_Pitch1.27mm, F.Cu at (191.4, 55.2)
- added P4: CONN_01X02_FAN, 2kwMotorController:TERM_2P_2-5_1990009, F.Cu at (152.0, 99.4)
- added P5: CONN_01X08_DEBUG, Pin_Headers:Pin_Header_Straight_1x08, F.Cu at (190.8, 64.4)
- added P6: CONN_01X03_UART, 2kwMotorController:TERM_3P_2-5_1990012, F.Cu at (189.8, 35.8)
- added P7: CONN_01X03_CAN, 2kwMotorController:TERM_3P_2-5_1990012, F.Cu at (179.8, 35.8)
- added P8: CONN_01X05_ENCODER, 2kwMotorController:TERM_5P_2-5_1990038, F.Cu at (170.0, 35.6)
- added R38: 220, Resistors_SMD:R_0603, F.Cu at (290.6, 10.0)
- added R39: 2.2k, Resistors_SMD:R_0603, F.Cu at (288.2, 14.4)
- added R40: 2.2k, Resistors_SMD:R_0603, F.Cu at (290.8, 14.4)
- added R41: 100, Resistors_SMD:R_0603, F.Cu at (293.2, 10.0)
- added R42: 10k, Resistors_SMD:R_0603, F.Cu at (295.8, 10.0)
- added R43: 220, Resistors_SMD:R_0603, F.Cu at (298.4, 10.0)
- added R44: 220, Resistors_SMD:R_0603, F.Cu at (304.0, 10.0)
- added R45: 220, Resistors_SMD:R_0603, F.Cu at (309.6, 10.0)
- added R46: 220, Resistors_SMD:R_0603, F.Cu at (272.6, 14.4)
- added R47: 0, Resistors_SMD:R_0603, F.Cu at (275.2, 14.4)
- added R48: 120, Resistors_SMD:R_0603, F.Cu at (277.6, 14.4)
- added R50: 100, Resistors_SMD:R_0603, F.Cu at (280.2, 14.4)
- added R51: 33, Resistors_SMD:R_0603, F.Cu at (282.8, 14.4)
- added R52: 100, Resistors_SMD:R_0603, F.Cu at (285.6, 14.4)
- added R54: 2.2k, Resistors_SMD:R_0603, F.Cu at (293.4, 14.4)
- added SW1: SW-SPST, 2kwMotorController:SW_SPST, F.Cu at (189.4, 105.2)
- added SW2: SW_PUSH, Buttons_Switches_ThroughHole:SW_PUSH_SMALL, F.Cu at (187.8, 43.6)
- added U21: 74LVCH2T45, 2kwMotorController:VSSOP8, F.Cu at (165.2, 41.6)
- added U8: PDM1-S, 2kwMotorController:PDM2-S, F.Cu at (150.8, 71.2)
- Q3, Q4, Q5, Q6, Q7, Q8: footprint TO_SOT_Packages_THT:TO-247_Horizontal_Neutral123_MountFromLS_largePads -> 2kwMotorController:TO-247_Horizontal_Neutral123_MountFromLS_largePads
- R14: value 1.8k -> 2.2k
- U11: footprint Housings_QFP:TQFP-128_14x14mm_Pitch0.4mm -> 2kwMotorController:TQFP-128_14x14mm_Pitch0.4mm_LONG
- moved C46 337.3 mm to (303.0, -16.5), turned to 0 degrees
- moved R37 332.4 mm to (300.0, -5.50), turned to 0 degrees
- moved D6 326.7 mm to (303.5, 22.0), turned to 0 degrees
- moved R36 325.3 mm to (297.5, -5.50), turned to 0 degrees
- moved R33 319.0 mm to (290.0, -5.50), turned to 0 degrees
- moved R35 305.8 mm to (295.0, -5.50), turned to 0 degrees
- moved R28 303.0 mm to (277.5, -5.50), turned to 0 degrees
- moved R32 301.9 mm to (287.5, -5.50), turned to 0 degrees
- moved C50 268.8 mm to (332.5, -13.0)
- moved C43 267.6 mm to (297.0, -16.5)
- moved R22 266.8 mm to (303.5, -11.0)
- moved R24 265.9 mm to (308.5, -11.0)
- moved C45 261.8 mm to (309.0, 4.50)
- moved C44 259.3 mm to (300.0, -16.5)
- moved C37 255.1 mm to (327.5, -7.00)
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Connections:
- C14 pad 2: GNDPWR -> GND
- C51 pad 1: +3V3 -> Net-(C51-Pad1)
- R9 pad 1: +BATT -> Net-(Q1-Pad4)
- R9 pad 2: Net-(Q1-Pad4) -> Net-(R9-Pad2)
- U18 pad 3: +3V3 -> Net-(C51-Pad1)
Routing:
- net GNDPWR: track 123.7 -> 165.7 mm, vias 0 -> 1
- net /h-bridge/I_SENSE+: track 85.6 -> 45.8 mm
- net /h-bridge/VBUS: track 88.9 -> 115.1 mm
- net /h-bridge/I_SENSE-: track 0.00 -> 23.4 mm
- net /h-bridge/BRAKE: track 0.00 -> 22.5 mm
- net /h-bridge/M-: track 85.6 -> 66.5 mm
- net GNDMBAT: track 30.5 -> 23.5 mm
- net Net-(C34-Pad2): track 43.8 -> 39.7 mm
- net GND: track 0.00 -> 2.28 mm
- added copper zone on In2.Cu, net +3V3
- added copper zone on In1.Cu, net GND
- added copper zone on In1.Cu, net GNDPWR
Other:
- board size 170.2 x 81.3 mm -> 160 x 81.5 mm
- rule pad_to_mask_clearance: 0.2 -> 0
- board text added: "BRK"
- board text added: "M+"
- board text added: "M-"

Commit message: H-bridge decoupling, footprints, mechanical
- Finished H-bridge decoupling study and chose H-bridge caps
- Changed LT3471 inductors to those found in reference design,
  made footprints for them
- Swapped Si86xx isolator for Si80xx (smaller package)
- Updated heatsink footprint with correct screw sizes
- Created mechanical hole footprints (M3, M4 screws)
Parts:
- removed JP3, JP4: Jumper_NO_Small, Pin_Headers:Pin_Header_Straight_1x02
- removed P8: CONN_01X05_ENCODER, 2kwMotorController:TERM_5P_2-5_1990038
- added C66: 1u, Capacitors_SMD:C_1206, F.Cu at (296.9, -22.5)
- added C67: 1u, Capacitors_SMD:C_0603, F.Cu at (299.9, -22.5)
- added C68: 1u, Capacitors_SMD:C_1206, F.Cu at (215.9, 61.5)
- added C69: 100n, Capacitors_SMD:C_0603, F.Cu at (218.4, 68.1)
- added C70: 100n, Capacitors_SMD:C_0603, F.Cu at (220.5, 75.2)
- added C71: 10u, Capacitors_SMD:C_0603, F.Cu at (213.4, 68.6)
- added D13: S210F, Diodes_SMD:SOD-123, F.Cu at (208.8, 62.5)
- added D14: S210F, Diodes_SMD:SOD-123, F.Cu at (208.3, 67.6)
- added P3: CONN_01X08_DEBUG, Pin_Headers:Pin_Header_Straight_1x08, F.Cu at (190.5, 64.5)
- added R55: 10k, Resistors_SMD:R_0603, F.Cu at (213.9, 73.7)
- C10: value 4.7u -> 100n
- C11: value 56p -> 1u
- C12: value 4.7u -> 10u; footprint Capacitors_SMD:C_0603 -> Capacitors_SMD:C_1206
- C13, C19, C25, C26, C60: value 100n -> 1u
- C14, C43, C44: value 1u -> 100n
- C15: value 10u -> 56p; footprint Capacitors_SMD:C_1206 -> Capacitors_SMD:C_0603
- C16: value 2.2u -> 56p
- C20, C23: value 100n -> 2.2u
- C21: value 2.2u -> 1u
- C22: value 100n -> 300p
- C24: value 1u -> 2.2u
- C27: footprint Capacitors_SMD:C_0603 -> Capacitors_SMD:C_1206
- C28, C61, C64, C65: value 100n -> 1u; footprint Capacitors_SMD:C_0603 -> Capacitors_SMD:C_1206
- C31: value 10p -> 100n
- C32: value 10p -> 10u
- C33: value 47n -> 10u
- C34: value 1.5m -> 2.2u; footprint Capacitors_ThroughHole:C_Radial_D18_L36_P7.5 -> Capacitors_SMD:C_0603
- C35: value 1.5m -> 100n; footprint Capacitors_ThroughHole:C_Radial_D18_L36_P7.5 -> Capacitors_SMD:C_0603
- C36, C55: value 10u -> 100n; footprint Capacitors_SMD:C_1206 -> Capacitors_SMD:C_0603
- C37: value 10u -> 1u; footprint Capacitors_SMD:C_1206 -> Capacitors_SMD:C_0603
- C4: value 1u -> 47n
- C40: value 10u -> 100n
- C46: value 10u -> 10p
- C47: value 300p -> 10p
- C49: value 1u -> 10n
- C5: value 4.7u -> 47n
- C50: footprint Capacitors_SMD:C_1206 -> Capacitors_SMD:C_0603
- C51: value 100n -> 1.5m; footprint Capacitors_SMD:C_0603 -> Capacitors_ThroughHole:C_Radial_D18_L36_P7.5
- C52: value 1u -> 1.5m; footprint Capacitors_SMD:C_0603 -> Capacitors_ThroughHole:C_Radial_D18_L36_P7.5
- C53: value 10n -> 100n
- C54: value 100n -> 10u
- C56: value 10u -> 1u
- C57, C58: value 47n -> 100n
- C6: value 100n -> 47n
- C62: value 2.2u -> 1u; footprint Capacitors_SMD:C_0603 -> Capacitors_SMD:C_1206
- C63: value 2.2u -> 100n
- C8: value 100n -> 4.7u
- C9: value 56p -> 100n
- D3: value LED -> MBRM-120
- D4: value MBRM-120 -> LED
- D6, D7: value S210F -> LED
- D8: value LED -> D
- L1: footprint Capacitors_SMD:C_0603 -> 2kwMotorController:INDUCTOR_NR40xx
- L2, L3: value 10u -> 15u; footprint Capacitors_SMD:C_0603 -> 2kwMotorController:INDUCTOR_NR40xx
- P2: value CONN_02X05_JTAG -> CONN_01X02_FAN; footprint Pin_Headers:Pin_Header_Straight_2x05_Pitch1.27mm -> 2kwMotorController:TERM_2P_2-5_1990009
- P4: value CONN_01X02_FAN -> CONN_02X05_JTAG; footprint 2kwMotorController:TERM_2P_2-5_1990009 -> Pin_Headers:Pin_Header_Straight_2x05_Pitch1.27mm
- P5: value CONN_01X08_DEBUG -> CONN_01X03_UART; footprint Pin_Headers:Pin_Header_Straight_1x08 -> 2kwMotorController:TERM_3P_2-5_1990012
- P6: value CONN_01X03_UART -> CONN_01X03_CAN
- P7: value CONN_01X03_CAN -> CONN_01X05_ENCODER; footprint 2kwMotorController:TERM_3P_2-5_1990012 -> 2kwMotorController:TERM_5P_2-5_1990038
- Q4: value IRFP4468 -> DMT10H010LK3; footprint 2kwMotorController:TO-247_Horizontal_Neutral123_MountFromLS_largePads -> TO_SOT_Packages_SMD:TO-252-2Lead
- Q9: value DMT10H010LK3 -> IRFP4468; footprint TO_SOT_Packages_SMD:TO-252-2Lead -> 2kwMotorController:TO-247_Horizontal_Neutral123_MountFromLS_largePads
- R1: value 270k -> 1.2M
- R10: value 110k -> 100k
- R11, R12, R24, R26, R7: value 10k -> 100
- R13: value 120k -> 10k
- R14, R40, R54: value 2.2k -> 10k
- R15, R27, R28, R29, R30: value 10k -> 220
- R16: value 4.87k -> 110k
- R17, R41, R50, R52: value 100 -> 10k
- R18, R4: value 470 -> 10k
- R19: value 10k -> 120k
- R2: value 100k -> 470
- R20: value 1k -> 2.2k
- R21: value 1 -> 2.2k
- R22, R23: value 2.2 -> 2.2k
- R3: value 1.2M -> 59.0
- R31: value 10k -> 0
- R32: value 2.2 -> 120
- R33: value 2.2 -> 470
- R34: value 2.2 -> 10k
- R35: value 2.2 -> 1k
- R36: value 10k -> 4.87k
- R38: value 220 -> 1
- R39: value 2.2k -> 2.2
- R42: value 10k -> 2.2
- R43, R46: value 220 -> 2.2
- R44, R45: value 220 -> 10k
- R47: value 0 -> 2.2
- R48: value 120 -> 2.2
- R5: value 59.0 -> 10k
- R51: value 33 -> 10k
- R6: value 10k -> 39k
- R8: value 39k -> 33
- R9: value 100 -> 270k
- U10: value LF33ABDT -> MCP1501T-30E; footprint TO_SOT_Packages_SMD:TO-252-2Lead -> TO_SOT_Packages_SMD:SOT-23-6
- U11: value TM4C1294KCPDT -> PDM1-S; footprint 2kwMotorController:TQFP-128_14x14mm_Pitch0.4mm_LONG -> 2kwMotorController:PDM2-S
- U12: value Si8640 -> MIC5225-5.0; footprint Housings_SOIC:SOIC-16_7.5x10.3mm_Pitch1.27mm -> TO_SOT_Packages_SMD:SOT-23-5
- U13: value MIC4127 -> TM4C1294KCPDT; footprint Housings_SOIC:SOIC-8_3.9x4.9mm_Pitch1.27mm -> 2kwMotorController:TQFP-128_14x14mm_Pitch0.4mm_LONG
- U14: value LM5102 -> 74LVCH2T45; footprint Housings_SSOP:MSOP-10_3x3mm_Pitch0.5mm -> 2kwMotorController:VSSOP8
- U15: value LM5102 -> SN65HVD231D; footprint Housings_SSOP:MSOP-10_3x3mm_Pitch0.5mm -> Housings_SOIC:SOIC-8_3.9x4.9mm_Pitch1.27mm
- U16: value MCP1501T-30E -> Si8045AA; footprint TO_SOT_Packages_SMD:SOT-23-6 -> Housings_SSOP:QSOP-16_3.9x4.9mm_Pitch0.635mm
- U17: value MIC5225-5.0 -> MIC4127; footprint TO_SOT_Packages_SMD:SOT-23-5 -> Housings_SOIC:SOIC-8_3.9x4.9mm_Pitch1.27mm
- U18: value SN65HVD231D -> MIC4127
- U19: value MIC4127 -> LM5102; footprint Housings_SOIC:SOIC-8_3.9x4.9mm_Pitch1.27mm -> Housings_SSOP:MSOP-10_3x3mm_Pitch0.5mm
- U2: value MCP6001 -> LAH-100P; footprint TO_SOT_Packages_SMD:SC-70-5 -> 2kwMotorController:LAH_100-P
- U20: value Si8640 -> Si8045AA; footprint Housings_SOIC:SOIC-16_7.5x10.3mm_Pitch1.27mm -> Housings_SSOP:QSOP-16_3.9x4.9mm_Pitch0.635mm
- U21: value 74LVCH2T45 -> LM5102; footprint 2kwMotorController:VSSOP8 -> Housings_SSOP:MSOP-10_3x3mm_Pitch0.5mm
- U3: value LAH-100P -> LOC110; footprint 2kwMotorController:LAH_100-P -> Housings_DIP:DIP-8_W7.62mm
- U4: value LOC110 -> MCP6001; footprint Housings_DIP:DIP-8_W7.62mm -> TO_SOT_Packages_SMD:SC-70-5
- U5: value MCP6001 -> ADA4805-1; footprint TO_SOT_Packages_SMD:SC-70-5 -> TO_SOT_Packages_SMD:SOT-23-6
- U6: value ADA4805-1 -> MCP6001; footprint TO_SOT_Packages_SMD:SOT-23-6 -> TO_SOT_Packages_SMD:SC-70-5
- U7: value LT3471 -> MIC5225-5.0; footprint Housings_DFN_QFN:DFN-10-1EP_3x3mm_Pitch0.5mm -> TO_SOT_Packages_SMD:SOT-23-5
- U8: value PDM1-S -> LT3471; footprint 2kwMotorController:PDM2-S -> Housings_DFN_QFN:DFN-10-1EP_3x3mm_Pitch0.5mm
- U9: value MIC5225-5.0 -> LF33ABDT; footprint TO_SOT_Packages_SMD:SOT-23-5 -> TO_SOT_Packages_SMD:TO-252-2Lead
- moved C51 208.0 mm to (68.1, 45.7)
- moved C34 195.4 mm to (262.1, 22.9)
- moved L3 173.9 mm to (171.8, 91.6), turned to 180 degrees
- moved C52 172.9 mm to (106.7, 45.7), turned to 180 degrees
- moved L1 164.7 mm to (174.1, 87.2)
- moved L2 163.7 mm to (181.2, 90.1), turned to 270 degrees
- moved C35 162.9 mm to (268.2, 25.9)
- moved U18 152.8 mm to (27.2, 68.8)
- moved U13 140.1 mm to (164.1, 62.0)
- moved U17 111.2 mm to (27.4, 76.5)
- moved U15 108.0 mm to (179.6, 46.2)
- moved U14 70.2 mm to (170.9, 46.0)
- moved U21 65.7 mm to (105.4, 68.8), turned to 90 degrees
- moved Q5 61.0 mm to (57.0, 64.0)
- moved P4 58.4 mm to (191.5, 56.4)
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Connections:
- C10 pad 1: GND -> +BATT
- C10 pad 2: -12V -> GND
- C11 pad 1: -12V -> +5V
- C11 pad 2: Net-(C11-Pad2) -> GND
- C12 pad 1: +12V -> +3V3
- C13 pad 1: +BATT -> Net-(C13-Pad1)
- C13 pad 2: GND -> Net-(C13-Pad2)
- C14 pad 1: +5V -> GND
- C14 pad 2: GND -> Net-(C14-Pad2)
- C15 pad 1: +3V3 -> +12V
- C15 pad 2: GND -> Net-(C15-Pad2)
- C16 pad 1: +3V3 -> -12V
- C17 pad 1: +3V3 -> GND
- C17 pad 2: GND -> -12V
- C18 pad 1: +3V3 -> +12V
- C19 pad 1: +3V3 -> GND
- C19 pad 2: GND -> -12V
- C20 pad 2: GND -> Net-(C20-Pad2)
- C21 pad 1: Net-(C21-Pad1) -> +12V
- C22 pad 2: GND -> GNDA
- C23 pad 1: +3V3 -> +12V
- C24 pad 1: Net-(C21-Pad1) -> +12V_ISO
- C24 pad 2: GND -> GNDPWR
- C25 pad 1: +3V3 -> +12V_ISO
- C25 pad 2: GND -> GNDPWR
- C26 pad 1: +3V3 -> +5V_ISO
- C26 pad 2: GND -> GNDPWR
- C27 pad 1: Net-(C21-Pad1) -> +12V
- C28 pad 1: +3V3 -> +12V
- C30 pad 1: Net-(C21-Pad1) -> Net-(C30-Pad1)
- C31 pad 1: Net-(C31-Pad1) -> +5V
- C32 pad 1: Net-(C32-Pad1) -> +3V3
- C33 pad 1: /mcu/VBUS_MOTOR -> +3V3
- C34 pad 1: /h-bridge/VBUS -> Net-(C34-Pad1)
- C34 pad 2: Net-(C34-Pad2) -> GND
- C35 pad 1: /h-bridge/VBUS -> +3V3
- C35 pad 2: Net-(C34-Pad2) -> GND
- C36 pad 1: /h-bridge/VBUS -> +3V3
- C36 pad 2: GNDPWR -> GND
- C37 pad 1: /h-bridge/VBUS -> Net-(C34-Pad1)
- C37 pad 2: GNDPWR -> GND
- C39 pad 1: +5V_ISO -> +3V3
- C39 pad 2: GNDPWR -> GND
- C4 pad 1: +BATT -> /mcu/VBUS_MOTOR
- C40 pad 1: +12V_ISO -> Net-(C34-Pad1)
- C40 pad 2: GNDPWR -> GND
- C41 pad 1: +12V_ISO -> +3V3
- C41 pad 2: GNDPWR -> GND
- C42 pad 1: +12V_ISO -> +3V3
- C42 pad 2: GNDPWR -> GND
- C43 pad 1: Net-(C43-Pad1) -> Net-(C34-Pad1)
- C43 pad 2: Net-(C43-Pad2) -> GND
- C44 pad 1: Net-(C44-Pad1) -> +3V3
- C44 pad 2: Net-(C44-Pad2) -> GND
- C45 pad 1: +12V_ISO -> +3V3
- C45 pad 2: GNDPWR -> GND
- C46 pad 1: +12V_ISO -> Net-(C46-Pad1)
- C46 pad 2: GNDPWR -> GND
- C47 pad 1: +3V3 -> Net-(C47-Pad1)
- C47 pad 2: GNDA -> GND
- C48 pad 1: +12V_ISO -> +3V3
- C48 pad 2: GNDPWR -> GNDA
- C49 pad 1: +5V_ISO -> +3V3
- C49 pad 2: GNDPWR -> GNDA
- C5 pad 1: +BATT -> /mcu/I_SENSOR_OUT
- C50 pad 1: +12V -> +3V3
- C51 pad 1: Net-(C51-Pad1) -> /h-bridge/VBUS
- C51 pad 2: GND -> Net-(C51-Pad2)
- C52 pad 1: +3V3 -> /h-bridge/VBUS
- C52 pad 2: GNDA -> Net-(C51-Pad2)
- C53 pad 1: +3V3 -> +5V_ISO
- C53 pad 2: GNDA -> GNDPWR
- C55 pad 1: /h-bridge/VBUS -> +12V_ISO
- C57 pad 1: /mcu/I_SENSOR_OUT -> +12V_ISO
- C57 pad 2: GND -> GNDPWR
- C58 pad 1: /mcu/VBAT_CTRL -> +12V_ISO
- C58 pad 2: GND -> GNDPWR
- C59 pad 1: +12V -> /h-bridge/VBUS
- C59 pad 2: GND -> GNDPWR
- C6 pad 1: Net-(C6-Pad1) -> /mcu/VBAT_CTRL
- C60 pad 1: +3V3 -> Net-(C60-Pad1)
- C60 pad 2: GND -> Net-(C60-Pad2)
- C61 pad 1: +5V_ISO -> /h-bridge/VBUS
- C62 pad 1: +12V -> /h-bridge/VBUS
- C62 pad 2: GND -> GNDPWR
- C63 pad 1: +12V_ISO -> +3V3
- C63 pad 2: GNDPWR -> GND
- C64 pad 1: +3V3 -> /h-bridge/VBUS
- C64 pad 2: GND -> GNDPWR
- C65 pad 1: +5V -> /h-bridge/VBUS
- C65 pad 2: GND -> GNDPWR
- C7 pad 1: Net-(C7-Pad1) -> +BATT
- C7 pad 2: Net-(C7-Pad2) -> GND
- C8 pad 1: GND -> +BATT
- C8 pad 2: Net-(C8-Pad2) -> GND
- C9 pad 1: +12V -> Net-(C9-Pad1)
- C9 pad 2: Net-(C9-Pad2) -> GND
- D1 pad 1: +12V -> +BATT
- D1 pad 2: Net-(D1-Pad2) -> +3V3
- D2 pad 1: GND -> +12V
- D2 pad 2: Net-(C7-Pad1) -> Net-(D2-Pad2)
- D3 pad 1: Net-(D3-Pad1) -> GND
- D3 pad 2: +12V_ISO -> Net-(C13-Pad1)
- D4 pad 1: +BATT -> Net-(D4-Pad1)
- D5 pad 2: +3V3 -> +12V
- D6 pad 1: Net-(C43-Pad2) -> Net-(D6-Pad1)
- D6 pad 2: GNDPWR -> GND
- D7 pad 1: Net-(C44-Pad2) -> Net-(D7-Pad1)
- D7 pad 2: GNDPWR -> +12V_ISO
- D8 pad 1: Net-(D8-Pad1) -> +12V
- D8 pad 2: +12V -> Net-(D8-Pad2)
- D9 pad 2: GND -> /mcu/LED_0
- L1 pad 2: Net-(D1-Pad2) -> Net-(D2-Pad2)
- L2 pad 2: Net-(C7-Pad2) -> Net-(C13-Pad2)
- L3 pad 1: Net-(C7-Pad1) -> Net-(C13-Pad1)
- P2 pad 1: Net-(P2-Pad1) -> +12V
- P2 pad 2: /mcu/JTAG_TMS -> Net-(D8-Pad2)
- P4 pad 1: +12V -> Net-(P4-Pad1)
- P4 pad 2: Net-(D10-Pad2) -> /mcu/JTAG_TMS
- P5 pad 1: /mcu/DEBUG_0 -> GND
- P5 pad 2: /mcu/DEBUG_1 -> /mcu/MCU_UART_RX
- P5 pad 3: /mcu/DEBUG_2 -> /mcu/MCU_UART_TX
- P6 pad 1: GND -> Net-(P6-Pad1)
- P6 pad 2: /mcu/MCU_UART_RX -> Net-(P6-Pad2)
- P6 pad 3: /mcu/MCU_UART_TX -> GND
- P7 pad 1: Net-(P7-Pad1) -> GND
- P7 pad 2: Net-(P7-Pad2) -> GND
- P7 pad 3: GND -> /mcu/ENCODER_CHA
- Q2 pad 5: Net-(D10-Pad2) -> Net-(D8-Pad2)
- Q2 pad 6: Net-(D10-Pad2) -> Net-(D8-Pad2)
- Q2 pad 7: Net-(D10-Pad2) -> Net-(D8-Pad2)
- Q2 pad 8: Net-(D10-Pad2) -> Net-(D8-Pad2)
- Q4 pad 2: /h-bridge/BRAKE -> Net-(C51-Pad2)
- Q5 pad 2: /h-bridge/VBUS -> /h-bridge/BRAKE
- Q5 pad 3: /h-bridge/I_SENSE+ -> GNDPWR
- Q6 pad 2: /h-bridge/I_SENSE+ -> /h-bridge/VBUS
- Q6 pad 3: GNDPWR -> /h-bridge/I_SENSE+
- Q7 pad 2: /h-bridge/VBUS -> /h-bridge/I_SENSE+
- Q7 pad 3: /h-bridge/M- -> GNDPWR
- Q8 pad 2: /h-bridge/M- -> /h-bridge/VBUS
- Q8 pad 3: GNDPWR -> /h-bridge/M-
- Q9 pad 2: Net-(C34-Pad2) -> /h-bridge/M-
- R1 pad 1: +9V -> Net-(C1-Pad2)
- R1 pad 2: Net-(R1-Pad2) -> /h-bridge/VBUS
- R10 pad 1: +12V -> Net-(R10-Pad1)
- R10 pad 2: Net-(C9-Pad2) -> GND
- R11 pad 1: GND -> /mcu/VBAT_CTRL
- R11 pad 2: Net-(C9-Pad2) -> Net-(R11-Pad2)
- R12 pad 1: Net-(C8-Pad2) -> Net-(Q1-Pad4)
- R12 pad 2: Net-(C11-Pad2) -> Net-(R12-Pad2)
- R13 pad 1: Net-(C11-Pad2) -> GND
- R13 pad 2: -12V -> Net-(Q1-Pad4)
- R14 pad 1: Net-(D3-Pad1) -> Net-(C9-Pad1)
- R14 pad 2: GNDPWR -> +BATT
- R15 pad 1: Net-(C6-Pad1) -> Net-(D4-Pad1)
- R15 pad 2: +BATT -> GND
- R16 pad 1: GND -> +12V
- R16 pad 2: Net-(R16-Pad2) -> Net-(C15-Pad2)
- R17 pad 1: +3V3 -> GND
- R17 pad 2: Net-(P2-Pad1) -> Net-(C15-Pad2)
- R18 pad 1: Net-(R18-Pad1) -> Net-(C14-Pad2)
- R18 pad 2: GND -> Net-(C16-Pad2)
- R19 pad 1: +3V3 -> Net-(C16-Pad2)
- R19 pad 2: /mcu/JTAG_RST_N -> -12V
- R2 pad 1: Net-(R1-Pad2) -> Net-(R2-Pad1)
- R2 pad 2: GND -> Net-(C1-Pad1)
- R20 pad 1: Net-(C31-Pad1) -> Net-(D5-Pad1)
- R20 pad 2: Net-(R20-Pad2) -> GND
- R21 pad 1: /h-bridge/VBUS -> Net-(D6-Pad1)
- R21 pad 2: /h-bridge/BRAKE -> -12V
- R22 pad 1: Net-(R22-Pad1) -> +12V_ISO
- R22 pad 2: Net-(Q9-Pad1) -> GNDPWR
- R23 pad 1: Net-(R23-Pad1) -> Net-(D7-Pad1)
- R23 pad 2: Net-(Q4-Pad1) -> GNDPWR
- R24 pad 1: Net-(R24-Pad1) -> Net-(Q2-Pad4)
- R24 pad 2: GNDPWR -> /power/PWM_FAN
- R25 pad 1: Net-(R25-Pad1) -> GND
- R25 pad 2: GNDPWR -> Net-(Q2-Pad4)
- R26 pad 1: /h-bridge/VBUS_EN_GD -> +3V3
- R26 pad 2: GNDPWR -> Net-(P4-Pad1)
- R27 pad 1: /h-bridge/VBUS_DIS_GD -> GND
- R27 pad 2: GNDPWR -> Net-(D9-Pad1)
- R28 pad 1: /h-bridge/PWM4_GD -> GND
- R28 pad 2: GNDPWR -> Net-(D10-Pad1)
- R29 pad 1: /h-bridge/PWM3_GD -> GND
- R29 pad 2: GNDPWR -> Net-(D11-Pad1)
- R3 pad 1: Net-(C1-Pad2) -> Net-(C2-Pad1)
- R3 pad 2: /h-bridge/VBUS -> GND
- R30 pad 1: /h-bridge/PWM2_GD -> GND
- R30 pad 2: GNDPWR -> Net-(D12-Pad1)
- R31 pad 1: /h-bridge/PWM1_GD -> Net-(R31-Pad1)
- R31 pad 2: GNDPWR -> GND
- R32 pad 1: Net-(Q6-Pad1) -> Net-(P6-Pad1)
- R32 pad 2: Net-(R32-Pad2) -> Net-(P6-Pad2)
- R33 pad 1: /h-bridge/I_SENSE+ -> Net-(R33-Pad1)
- R33 pad 2: Net-(C43-Pad2) -> GND
- R34 pad 1: /h-bridge/M- -> +3V3
- R34 pad 2: Net-(C44-Pad2) -> /mcu/JTAG_RST_N
- R35 pad 1: Net-(Q8-Pad1) -> Net-(C46-Pad1)
- R36 pad 1: Net-(R36-Pad1) -> GND
- R36 pad 2: GNDPWR -> Net-(R36-Pad2)
- R37 pad 1: Net-(R37-Pad1) -> /h-bridge/VBUS_EN_GD
- R38 pad 1: Net-(D5-Pad1) -> /h-bridge/VBUS
- R38 pad 2: GND -> /h-bridge/BRAKE
- R39 pad 1: Net-(D8-Pad1) -> Net-(R39-Pad1)
- R39 pad 2: GND -> Net-(Q4-Pad1)
- R4 pad 2: Net-(C1-Pad1) -> +3V3
- R40 pad 1: Net-(D9-Pad1) -> /h-bridge/VBUS_DIS_GD
- R40 pad 2: -12V -> GNDPWR
- R41 pad 1: Net-(Q2-Pad4) -> /h-bridge/VBUS_ST_GD
- R41 pad 2: /power/PWM_FAN -> GNDPWR
- R42 pad 1: GND -> Net-(R42-Pad1)
- R42 pad 2: Net-(Q2-Pad4) -> Net-(Q5-Pad1)
- R43 pad 1: GND -> Net-(R43-Pad1)
- R43 pad 2: Net-(D11-Pad1) -> Net-(Q3-Pad1)
- R44 pad 1: GND -> Net-(R44-Pad1)
- R44 pad 2: Net-(D12-Pad1) -> GNDPWR
- R45 pad 1: GND -> Net-(R45-Pad1)
- R45 pad 2: Net-(D13-Pad1) -> GNDPWR
- R46 pad 1: GND -> Net-(Q7-Pad1)
- R46 pad 2: Net-(D14-Pad1) -> Net-(R46-Pad2)
- R47 pad 1: Net-(R47-Pad1) -> /h-bridge/I_SENSE+
- R47 pad 2: GND -> Net-(C60-Pad2)
- R48 pad 1: Net-(P7-Pad1) -> /h-bridge/M-
- R48 pad 2: Net-(P7-Pad2) -> Net-(C67-Pad2)
- R49 pad 1: Net-(R49-Pad1) -> Net-(Q9-Pad1)
- R49 pad 2: Net-(Q3-Pad1) -> Net-(R49-Pad2)
- R5 pad 1: Net-(C2-Pad1) -> Net-(R5-Pad1)
- R5 pad 2: GND -> Net-(C2-Pad1)
- R50 pad 1: /mcu/VBUS_MOTOR -> /h-bridge/PWM4_GD
- R50 pad 2: Net-(C3-Pad1) -> GNDPWR
- R51 pad 1: /mcu/I_SENSOR_OUT -> /h-bridge/PWM3_GD
- R51 pad 2: Net-(R51-Pad2) -> GNDPWR
- R52 pad 1: /mcu/VBAT_CTRL -> /h-bridge/PWM2_GD
- R52 pad 2: Net-(R52-Pad2) -> GNDPWR
- R53 pad 1: /h-bridge/VBUS_ST_GD -> Net-(R53-Pad1)
- R54 pad 1: +12V_ISO -> /h-bridge/PWM1_GD
- R6 pad 2: +3V3 -> Net-(C3-Pad2)
- R7 pad 1: Net-(R7-Pad1) -> /mcu/VBUS_MOTOR
- R7 pad 2: Net-(C2-Pad1) -> Net-(C3-Pad1)
- R8 pad 1: Net-(R8-Pad1) -> /mcu/I_SENSOR_OUT
- R8 pad 2: Net-(C3-Pad2) -> Net-(R8-Pad2)
- R9 pad 1: Net-(Q1-Pad4) -> +9V
- R9 pad 2: Net-(R9-Pad2) -> Net-(R10-Pad1)
- SW1 pad 2: Net-(R9-Pad2) -> Net-(R12-Pad2)
- SW2 pad 1: Net-(R18-Pad1) -> Net-(R33-Pad1)
- TH1 pad 1: Net-(C34-Pad2) -> Net-(C51-Pad2)
- U10 pad 1: +BATT -> +3V3
- U10 pad 2: GND -> Net-(U10-Pad2)
- U10 pad 3: +3V3 -> Net-(U10-Pad2)
- U11 pad 1: Net-(U11-Pad1) -> +12V
- U11 pad 2: Net-(U11-Pad2) -> GND
- U11 pad 4: Net-(U11-Pad4) -> GNDPWR
- U11 pad 6: Net-(U11-Pad6) -> +12V_ISO
- U12 pad 1: +3V3 -> +12V_ISO
- U12 pad 2: GND -> GNDPWR
- U12 pad 3: /h-bridge/VBUS_ST_MCU -> +12V_ISO
- U12 pad 4: /h-bridge/VBUS_DIS_MCU -> Net-(U12-Pad4)
- U12 pad 5: /h-bridge/VBUS_EN_MCU -> +5V_ISO
- U13 pad 2: /h-bridge/VBUS_DIS_GD -> Net-(U13-Pad2)
- U13 pad 3: GNDPWR -> Net-(U13-Pad3)
- U13 pad 4: /h-bridge/VBUS_ST_GD -> Net-(U13-Pad4)
- U13 pad 5: Net-(R22-Pad1) -> Net-(U13-Pad5)
- U13 pad 6: +12V_ISO -> Net-(U13-Pad6)
- U13 pad 7: Net-(R23-Pad1) -> +3V3
- U13 pad 8: Net-(U13-Pad8) -> +3V3
- U14 pad 1: +12V_ISO -> +3V3
- U14 pad 2: Net-(C43-Pad1) -> /mcu/QEI_PHA
- U14 pad 3: Net-(Q5-Pad1) -> /mcu/QEI_PHB
- U14 pad 4: Net-(C43-Pad2) -> GND
- U14 pad 5: Net-(R24-Pad1) -> GND
- U14 pad 6: Net-(R25-Pad1) -> /mcu/ENCODER_CHA
- U14 pad 7: /h-bridge/PWM1_GD -> /mcu/ENCODER_CHB
- U14 pad 8: /h-bridge/PWM2_GD -> +5V
- U15 pad 1: +12V_ISO -> /mcu/CAN_TX
- U15 pad 2: Net-(C44-Pad1) -> GND
- U15 pad 3: Net-(Q7-Pad1) -> Net-(C30-Pad1)
- U15 pad 4: Net-(C44-Pad2) -> /mcu/CAN_RX
- U15 pad 5: Net-(R37-Pad1) -> Net-(U15-Pad5)
- U15 pad 6: Net-(R36-Pad1) -> Net-(P6-Pad2)
- U15 pad 7: /h-bridge/PWM3_GD -> Net-(P6-Pad1)
- U15 pad 8: /h-bridge/PWM4_GD -> Net-(R31-Pad1)
- U16 pad 2: Net-(U16-Pad2) -> GND
- U16 pad 3: Net-(U16-Pad2) -> /h-bridge/VBUS_ST_MCU
- U16 pad 4: +3V3 -> /h-bridge/VBUS_DIS_MCU
- U16 pad 5: Net-(C16-Pad2) -> /h-bridge/VBUS_EN_MCU
- U16 pad 6: +3V3 -> GND
- U17 pad 1: +12V_ISO -> Net-(U17-Pad1)
- U17 pad 2: GNDPWR -> /h-bridge/VBUS_DIS_GD
- U17 pad 3: +12V_ISO -> GNDPWR
- U17 pad 4: Net-(U17-Pad4) -> /h-bridge/VBUS_ST_GD
- U17 pad 5: +5V_ISO -> Net-(R39-Pad1)
- U18 pad 1: /mcu/CAN_TX -> Net-(U18-Pad1)
- U18 pad 2: GND -> /h-bridge/VBUS_EN_GD
- U18 pad 3: Net-(C51-Pad1) -> GNDPWR
- U18 pad 4: /mcu/CAN_RX -> GNDPWR
- U18 pad 6: Net-(P7-Pad2) -> +12V_ISO
- U18 pad 7: Net-(P7-Pad1) -> Net-(R43-Pad1)
- U18 pad 8: Net-(R47-Pad1) -> Net-(U18-Pad8)
- U19 pad 1: Net-(U19-Pad1) -> +12V_ISO
- U19 pad 2: /h-bridge/VBUS_EN_GD -> Net-(C60-Pad1)
- U19 pad 3: GNDPWR -> Net-(Q6-Pad1)
- U19 pad 4: GNDPWR -> Net-(C60-Pad2)
- U19 pad 5: Net-(U19-Pad5) -> Net-(R44-Pad1)
- U19 pad 6: +12V_ISO -> Net-(R45-Pad1)
- U19 pad 7: Net-(R49-Pad1) -> /h-bridge/PWM1_GD
- U19 pad 8: Net-(U19-Pad8) -> /h-bridge/PWM2_GD
- U2 pad 1: Net-(R52-Pad2) -> /h-bridge/I_SENSE+
- U2 pad 2: +3.3VADC -> /h-bridge/I_SENSE-
- U2 pad 3: Net-(R1-Pad2) -> -12V
- U2 pad 4: Net-(R52-Pad2) -> +12V
- U2 pad 5: GND -> Net-(C2-Pad1)
- U20 pad 7: (no net) -> Net-(U20-Pad7)
- U21 pad 1: +3V3 -> +12V_ISO
- U21 pad 2: /mcu/QEI_PHA -> Net-(C67-Pad1)
- U21 pad 3: /mcu/QEI_PHB -> Net-(Q8-Pad1)
- U21 pad 4: GND -> Net-(C67-Pad2)
- U21 pad 5: GND -> Net-(R55-Pad1)
- U21 pad 6: /mcu/ENCODER_CHA -> Net-(R53-Pad1)
- U21 pad 7: /mcu/ENCODER_CHB -> /h-bridge/PWM3_GD
- U21 pad 8: +5V -> /h-bridge/PWM4_GD
- U3 pad 1: /h-bridge/I_SENSE+ -> Net-(R2-Pad1)
- U3 pad 2: /h-bridge/I_SENSE- -> +12V_ISO
- U3 pad 3: -12V -> Net-(C1-Pad2)
- U3 pad 4: +12V -> GNDPWR
- U3 pad 5: Net-(C2-Pad1) -> GND
- U4 pad 1: Net-(R4-Pad1) -> Net-(C3-Pad1)
- U4 pad 2: +12V_ISO -> GND
- U4 pad 3: Net-(C1-Pad2) -> GND
- U4 pad 4: GNDPWR -> Net-(C3-Pad2)
- U4 pad 5: GND -> +3.3VADC
- U5 pad 1: Net-(C3-Pad1) -> Net-(R8-Pad2)
- U5 pad 3: GND -> Net-(R5-Pad1)
- U5 pad 4: Net-(C3-Pad2) -> Net-(R8-Pad2)
- U6 pad 1: Net-(R51-Pad2) -> Net-(R11-Pad2)
- U6 pad 2: GND -> +3.3VADC
- U6 pad 3: Net-(R7-Pad1) -> Net-(R10-Pad1)
- U6 pad 4: Net-(R51-Pad2) -> Net-(R11-Pad2)
- U6 pad 5: +3.3VADC -> GND
- U7 pad 1: Net-(C9-Pad2) -> +BATT
- U7 pad 2: Net-(C8-Pad2) -> GND
- U7 pad 3: Net-(C8-Pad2) -> +BATT
- U7 pad 4: Net-(C11-Pad2) -> Net-(U7-Pad4)
- U7 pad 5: GND -> +5V
- U8 pad 1: +12V -> Net-(C15-Pad2)
- U8 pad 2: GND -> Net-(C14-Pad2)
- U8 pad 4: GNDPWR -> Net-(C16-Pad2)
- U8 pad 5: Net-(U8-Pad5) -> GND
- U8 pad 6: +12V_ISO -> Net-(C13-Pad2)
- U9 pad 3: +BATT -> +3V3
- Y1 pad 1: Net-(C32-Pad1) -> Net-(C47-Pad1)
- Y1 pad 2: Net-(C31-Pad1) -> Net-(C46-Pad1)
Routing:
- net /h-bridge/VBUS: track 115.1 -> 166.2 mm
- net Net-(C51-Pad2): track 0.00 -> 39.7 mm
- net Net-(C34-Pad2): track 39.7 -> 0.00 mm
- net /h-bridge/M-: track 66.5 -> 29.5 mm
- net GNDPWR: track 165.7 -> 190.7 mm
- net /h-bridge/I_SENSE+: track 45.8 -> 25.4 mm
- net /h-bridge/BRAKE: track 22.5 -> 6.00 mm

Commit message: Bulk cap layout, diodes, lugs, leds, trimpots
- Moved H-bridge bulk capacitors to horizontal layout
- Changed H-bridge and fan diodes to 100V schottky
- Made 4AWG lug mount footprint, added lugs to BOM
- Tweaked LED resistor values, added LEDs to BOM
- Made trimpot footprint, added trimpots to BOM
- Added snubber to ferrite bead circuit; also added FB to BOM
Parts:
- removed JP2: Jumper_NO_Small, Pin_Headers:Pin_Header_Straight_1x02
- removed R38: 1, Resistors_SMD:R_0603
- added C72: 1u, Capacitors_SMD:C_0603, F.Cu at (210.8, 54.0)
- added D10: LED, LEDs:LED_0603, F.Cu at (208.3, 41.3)
- added D11: LED, LEDs:LED_0603, F.Cu at (207.6, 46.4)
- added D12: LED, LEDs:LED_0603, F.Cu at (215.9, 50.2)
- added FB1: FERRITE_BEAD, Capacitors_SMD:C_0603, F.Cu at (228.6, 33.0)
- added M1: MOUNTING_HOLE, 2kwMotorController:M4-SCREW-HOLE, F.Cu at (44.0, 110.2)
- added M2: MOUNTING_HOLE, 2kwMotorController:M4-SCREW-HOLE, F.Cu at (130.0, 111.2)
- added M3: MOUNTING_HOLE, 2kwMotorController:M4-SCREW-HOLE, F.Cu at (46.8, 33.2)
- added M4: MOUNTING_HOLE, 2kwMotorController:M4-SCREW-HOLE, F.Cu at (124.2, 33.0)
- added M5: MOUNTING_HOLE, 2kwMotorController:M4-SCREW-HOLE, F.Cu at (156.5, 112.0)
- added M6: MOUNTING_HOLE, 2kwMotorController:M4-SCREW-HOLE, F.Cu at (143.5, 39.0)
- added P10: CONN_01_BRK, 2kwMotorController:M6_4AWG_LUG_TERM, F.Cu at (40.6, 69.2)
- added P11: CONN_01_M+, 2kwMotorController:M6_4AWG_LUG_TERM, F.Cu at (142.2, 109.2)
- added P12: CONN_01_M-, 2kwMotorController:M6_4AWG_LUG_TERM, F.Cu at (99.1, 108.6)
- added P8: CONN_01_V+, 2kwMotorController:M6_4AWG_LUG_TERM, F.Cu at (40.6, 54.6)
- added P9: CONN_01_V-, 2kwMotorController:M6_4AWG_LUG_TERM, F.Cu at (40.6, 83.2)
- added R56: 2.2, Resistors_SMD:R_0603, F.Cu at (209.6, 36.8)
- added R57: 2.2k, Resistors_SMD:R_0603, F.Cu at (215.3, 35.6)
- added R58: 2.2k, Resistors_SMD:R_0603, F.Cu at (224.8, 41.3)
- added RV1: 100, 2kwMotorController:Trimpot-23B, F.Cu at (224.2, 54.0)
- added RV2: 36k, 2kwMotorController:Trimpot-23B, F.Cu at (213.4, 42.5)
- C51, C52: value 1.5m -> 1m; footprint Capacitors_ThroughHole:C_Radial_D18_L36_P7.5 -> 2kwMotorController:Cap_Horizontal_D18_L36
- C61, C62, C64, C65: value 1u -> 10n
- D1, D2, D3: footprint Diodes_SMD:SOD-123 -> 2kwMotorController:DIODE_POWERMITE
- D13, D14: value S210F -> SK310-B; footprint Diodes_SMD:SOD-123 -> 2kwMotorController:DO-214AA
- D4, D5, D6, D7, D9: footprint Diodes_SMD:SOD-123 -> LEDs:LED_0603
- D8: value D -> MBRM-120; footprint Diodes_SMD:SOD-123 -> 2kwMotorController:DIODE_POWERMITE
- P5: footprint 2kwMotorController:TERM_3P_2-5_1990012 -> Pin_Headers:Pin_Header_Straight_1x03
- Q4: moved to B.Cu
- R15, R27, R28, R29, R30: value 220 -> 120
- R20, R21, R23: value 2.2k -> 1.8k
- U3: footprint Housings_DIP:DIP-8_W7.62mm -> SMD_Packages:DIP-8_SMD
- moved JP1 110.1 mm to (151.1, 33.7)
- moved C52 62.0 mm to (71.1, 96.5), turned to 0 degrees
- moved P3 47.4 mm to (157.5, 30.5), turned to 90 degrees
- moved P4 35.7 mm to (162.6, 35.6), turned to 270 degrees
- moved P2 28.8 mm to (182.9, 104.1), turned to 270 degrees
- moved Q4 24.3 mm to (72.1, 73.2), turned to 180 degrees
- moved P7 23.6 mm to (182.9, 55.2), turned to 270 degrees
- moved D7 20.0 mm to (322.6, 30.5)
- moved SW2 18.5 mm to (170.2, 38.1)
- moved Q1 18.3 mm to (162.6, 104.1)
- moved TH1 17.8 mm to (83.8, 17.8)
- moved U12 14.1 mm to (129.0, 64.5)
- moved SW1 13.1 mm to (188.0, 81.3)
- moved U14 10.9 mm to (160.0, 45.7)
- moved U3 8.86 mm to (150.4, 46.2), turned to 270 degrees
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Connections:
- C30 pad 1: Net-(C30-Pad1) -> +3V3
- JP1 pad 1: GND -> Net-(JP1-Pad1)
- JP1 pad 2: /mcu/CAN_ID_0 -> GND
- U13 pad 5: Net-(U13-Pad5) -> Net-(JP1-Pad1)
- U15 pad 3: Net-(C30-Pad1) -> +3V3
Routing:
- net GNDPWR: track 190.7 -> 110.9 mm, vias 1 -> 0
- net /h-bridge/M-: track 29.5 -> 66.5 mm
- net /h-bridge/VBUS: track 166.2 -> 140.8 mm, vias 0 -> 1
- net /h-bridge/I_SENSE+: track 25.4 -> 45.8 mm
- net /h-bridge/BRAKE: track 6.00 -> 23.5 mm
- net Net-(C51-Pad2): track 39.7 -> 50.8 mm
Other:
- board size 160 x 81.5 mm -> 160 x 88.5 mm

Commit message: Inrush circuit, mounting hole position, temp sensor
- Split inrush circuit (one for each bulk cap). Replaced NTC
  thermistor with 2W power resistor. Replaced D2Pak MOSFET with
  LFPAK MOSFETs.
- Approximate position of mechanical holes chosen.
- Added thermistor temp sensor circuits.
Parts:
- removed SW1: SW-SPST, 2kwMotorController:SW_SPST
- removed TH1: B57127P100M301, Resistors_ThroughHole:Resistor_Vertical_RM7.5mm
- added C73: 100n, Capacitors_SMD:C_0603, F.Cu at (266.4, 49.5)
- added C74: 100n, Capacitors_SMD:C_0603, F.Cu at (272.9, 41.3)
- added C75: 100n, Capacitors_SMD:C_0603, F.Cu at (275.1, 46.0)
- added C76: 100n, Capacitors_SMD:C_0603, F.Cu at (275.5, 51.3)
- added C77: 100n, Capacitors_SMD:C_0603, F.Cu at (260.9, 42.0)
- added C78: 100n, Capacitors_SMD:C_0603, F.Cu at (259.6, 47.0)
- added C79: 100n, Capacitors_SMD:C_0603, F.Cu at (258.4, 51.6)
- added C80, C81: 47n, Capacitors_SMD:C_0603, F.Cu at (220.6, 89.5)
- added Q10: PSMN021-100, TO_SOT_Packages_SMD:SOT-669_LFPAK_ThermalVias-1, F.Cu at (62.0, 105.2)
- added R38: 10k, Resistors_SMD:R_0603, F.Cu at (266.3, 41.8)
- added R59, R62, R63: 10k, Resistors_SMD:R_0603, F.Cu at (220.6, 89.5)
- added R60, R61: 100, Resistors_SMD:R_0603, F.Cu at (220.6, 89.5)
- added R64: 150, 2kwMotorController:RESISTOR_FMP200, F.Cu at (69.8, 111.8)
- added R65: 150, 2kwMotorController:RESISTOR_FMP200, F.Cu at (68.6, 30.5)
- added U22, U23: MCP6001, TO_SOT_Packages_SMD:SC-70-5, F.Cu at (220.6, 89.5)
- D8: value MBRM-120 -> SK310-B
- Q4: value DMT10H010LK3 -> PSMN021-100; footprint TO_SOT_Packages_SMD:TO-252-2Lead -> TO_SOT_Packages_SMD:SOT-669_LFPAK_ThermalVias-1; moved to F.Cu
- R13: value 10k -> 100
- R39: value 2.2 -> 100
- moved M3 129.2 mm to (154.3, 104.8)
- moved M5 89.8 mm to (113.7, 33.0)
- moved M4 78.5 mm to (45.7, 33.7)
- moved Q4 40.1 mm to (59.6, 35.1), turned to 0 degrees
- moved U18 34.7 mm to (57.5, 52.1)
- moved U17 31.8 mm to (57.5, 86.6)
- moved M2 17.6 mm to (113.7, 104.8)
- moved JP1 15.3 mm to (165.1, 40.0), turned to 90 degrees
- moved M6 11.3 mm to (153.0, 33.0)
- moved P2 8.27 mm to (183.4, 112.4)
- moved P1 7.63 mm to (183.3, 104.1)
- moved P4 6.38 mm to (168.9, 34.9)
- moved P3 6.35 mm to (163.8, 30.5)
- moved M1 6.35 mm to (45.7, 104.1)
- moved SW2 5.12 mm to (175.3, 37.5)
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Connections:
- C2 pad 2: GND -> GNDA
- C4 pad 2: GND -> GNDA
- C5 pad 2: GND -> GNDA
- C52 pad 2: Net-(C51-Pad2) -> Net-(C52-Pad2)
- C6 pad 2: GND -> GNDA
- P7 pad 2: GND -> /mcu/ENCODER_INDEX
- Q4 pad 2: Net-(C51-Pad2) -> Net-(C52-Pad2)
- R12 pad 2: Net-(R12-Pad2) -> +BATT
- R13 pad 1: GND -> Net-(R13-Pad1)
- R13 pad 2: Net-(Q1-Pad4) -> Net-(Q10-Pad1)
- R3 pad 2: GND -> GNDA
- R6 pad 2: Net-(C3-Pad2) -> Net-(C3-Pad1)
- R7 pad 2: Net-(C3-Pad1) -> Net-(C3-Pad2)
- R9 pad 1: +9V -> +BATT
- RV2 pad 1: Net-(RV2-Pad1) -> Net-(R6-Pad1)
- RV2 pad 2: Net-(C3-Pad1) -> Net-(C3-Pad2)
- RV2 pad 3: Net-(R6-Pad1) -> Net-(RV2-Pad3)
- U18 pad 2: /h-bridge/VBUS_EN_GD -> /h-bridge/VBUS_ST_GD
- U18 pad 4: GNDPWR -> /h-bridge/VBUS_EN_GD
- U18 pad 5: Net-(U18-Pad5) -> Net-(R43-Pad1)
- U18 pad 7: Net-(R43-Pad1) -> Net-(R13-Pad1)
- U3 pad 5: GND -> GNDA
- U3 pad 6: Net-(C3-Pad2) -> Net-(C3-Pad1)
- U4 pad 1: Net-(C3-Pad1) -> Net-(C3-Pad2)
- U4 pad 2: GND -> GNDA
- U4 pad 3: GND -> GNDA
- U4 pad 4: Net-(C3-Pad2) -> Net-(C3-Pad1)
- U4 pad 5: +3.3VADC -> +3V3
- U5 pad 2: GND -> GNDA
- U5 pad 5: +3.3VADC -> +3V3
- U5 pad 6: +3.3VADC -> +3V3
- U6 pad 2: +3.3VADC -> +3V3
- U6 pad 5: GND -> GNDA
Routing:
- net /h-bridge/VBUS: track 140.8 -> 89.7 mm, vias 1 -> 0
- net Net-(C51-Pad2): track 50.8 -> 0.00 mm
- net /h-bridge/I_SENSE+: track 45.8 -> 56.7 mm
- net GNDPWR: track 110.9 -> 101.3 mm
- net /h-bridge/I_SENSE-: track 23.4 -> 27.3 mm
- net /h-bridge/BRAKE: track 23.5 -> 22.2 mm
- net /h-bridge/M-: track 66.5 -> 65.9 mm

Commit message: High amp routes, sensors
- Adjusted high current routing to improve clearances. Recommend
  3mm high busbar to compensate for reduced busbar width to 2mm.
- Shrank TO-247 pads by 1mm (lengthwise) to improve busbar clearance.
- Removed unecessary buffers / SAR ADC drive circuits from low-bandwidth
  sensors.
Parts:
- removed C73, C78, C79: 100n, Capacitors_SMD:C_0603
- removed C80, C81: 47n, Capacitors_SMD:C_0603
- removed R11, R60, R61: 100, Resistors_SMD:R_0603
- removed U22, U23, U6: MCP6001, TO_SOT_Packages_SMD:SC-70-5
- C6: value 47n -> 100n
- moved Q2 63.4 mm to (234.7, 93.0)
- moved L1 48.5 mm to (220.3, 101.9)
- moved L2 48.5 mm to (227.4, 104.8)
- moved U10 48.5 mm to (230.3, 98.1)
- moved U8 48.5 mm to (222.0, 107.2)
- moved L3 48.5 mm to (218.0, 106.3)
- moved Q1 47.3 mm to (209.3, 97.0)
- moved U9 28.2 mm to (208.3, 82.8)
- moved U17 5.39 mm to (57.5, 92.0)
- moved P12 3.07 mm to (96.0, 109.5)
- moved M6 2.97 mm to (156.0, 33.0)
- moved M2 2.67 mm to (111.0, 105.0)
- moved M5 2.67 mm to (111.0, 33.0)
- moved U18 2.32 mm to (57.5, 49.8)
- moved M3 1.71 mm to (156.0, 105.0)
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Connections:
- C52 pad 1: /h-bridge/VBUS -> Net-(C52-Pad1)
- C52 pad 2: Net-(C52-Pad2) -> /h-bridge/VBUS
- C6 pad 2: GNDA -> GND
- C76 pad 1: Net-(C76-Pad1) -> /mcu/BRIDGE_TEMP
- C77 pad 1: Net-(C77-Pad1) -> /sensors/BRIDGE_TEMP
- Q4 pad 2: Net-(C52-Pad2) -> Net-(C52-Pad1)
- R10 pad 1: Net-(R10-Pad1) -> /mcu/VBAT_CTRL
- R38 pad 2: Net-(C76-Pad1) -> /mcu/BRIDGE_TEMP
- R59 pad 2: Net-(C77-Pad1) -> /sensors/BRIDGE_TEMP
- R65 pad 1: Net-(C52-Pad2) -> Net-(C52-Pad1)
- R9 pad 2: Net-(R10-Pad1) -> /mcu/VBAT_CTRL
Routing:
- net /h-bridge/VBUS: track 89.7 -> 84.4 mm
- net /h-bridge/I_SENSE+: track 56.7 -> 54.3 mm
- net /h-bridge/M-: track 65.9 -> 64.2 mm
- net /h-bridge/BRAKE: track 22.2 -> 20.9 mm
- net GNDMBAT: track 23.5 -> 24.0 mm
- net /h-bridge/I_SENSE-: track 27.3 -> 27.8 mm
Other:
- outline, holes or cut-outs redrawn
- board text added: "BRAKE"
- board text added: "GND"
- board text added: "MOTOR +"
- board text added: "MOTOR -"
- board text added: "VBUS"
- board text removed: "BRK"
- board text removed: "M+"
- board text removed: "M-"
