File: hardware/2kwMotorController.kicad_pcb (KiCad board)
At the start: 4 copper layers, 170 x 88 mm, 214 parts, among them M1 MOUNTING_HOLE, M2 MOUNTING_HOLE, M3 MOUNTING_HOLE, M4 MOUNTING_HOLE, M5 MOUNTING_HOLE, M6 MOUNTING_HOLE, P1 CONN_01X02_CBAT, P10 CONN_01_BRK, P11 CONN_01_M+, P12 CONN_01_M-, P13 CONN_01X02_MTMP, P14 CONN_01X02_BTMP, P2 CONN_01X02_FAN, P3 CONN_01X08_DEBUG, P4 CONN_02X05_JTAG, P5 CONN_01X03_UART, P6 CONN_01X03_CAN, P7 CONN_01X05_ENCODER, P8 CONN_01_V+, P9 CONN_01_V-, Q1 DMG4712SSS, Q10 PSMN021-100, Q2 DMG4712SSS, Q3 IRFP4468, Q4 PSMN021-100, Q5 IRFP4468, Q6 IRFP4468, Q7 IRFP4468, Q8 IRFP4468, Q9 IRFP4468, SW2 SW_PUSH, U1 LM358, U10 MCP1501T-30E, U11 PDM1-S, U12 MIC5225-5.0, U13 TM4C1294KCPDT, U14 74LVCH2T45, U15 SN65HVD231D, U16 Si8045AA, U17 MIC4127, U18 MIC4127, U19 LM5102, U2 LAH-100P, U20 Si8045AA, U21 LM5102, U3 LOC110, U4 MCP6001, U5 ADA4805-1, U7 MIC5225-5.0, U8 LT3471, U9 LF33ABDT, Y1 NX5032GA

Commit message: Gate driver layout mostly complete
- Gate driver layout
- Switch LM5102 for UCC27211 (higher current, more robust)
- Tweak gate drive circuit passives
- No soldermask on high-current traces
- Fix error in orientation of LAH-100P footprint
- Improved draft layout of control section
Parts:
- removed R44, R45, R50, R51, R52, R53, R54, R55: 10k, Resistors_SMD:R_0603
- removed U21: LM5102, Housings_SSOP:MSOP-10_3x3mm_Pitch0.5mm
- added C79: 1u, Capacitors_SMD:C_0603, F.Cu at (164.0, 74.0)
- added C80: 100n, Capacitors_SMD:C_0603, F.Cu at (111.0, 68.8)
- added C81: 100n, Capacitors_SMD:C_0603, F.Cu at (80.8, 68.8)
- added R11: 10k, Resistors_SMD:R_0603, F.Cu at (64.5, 78.5)
- added U6: UCC27211, Housings_SOIC:SOIC-8-1EP_3.9x4.9mm_Pitch1.27mm, F.Cu at (103.5, 69.5)
- C12: footprint Capacitors_SMD:C_1206 -> Capacitors_SMD:C_0805
- C17, C18, C32, C33: footprint Capacitors_SMD:C_0603 -> Capacitors_SMD:C_0805
- C23, C24, R22: moved to B.Cu
- C27, C28: footprint Capacitors_SMD:C_1206 -> Capacitors_SMD:C_0603
- C54, C71: value 10u -> 4.7u; footprint Capacitors_SMD:C_0603 -> Capacitors_SMD:C_0805
- U19: value LM5102 -> UCC27211; footprint Housings_SSOP:MSOP-10_3x3mm_Pitch0.5mm -> Housings_SOIC:SOIC-8-1EP_3.9x4.9mm_Pitch1.27mm
- moved R41 256.5 mm to (52.5, 98.5), turned to 180 degrees
- moved R40 247.7 mm to (47.8, 62.2), turned to 90 degrees
- moved R37 242.5 mm to (61.8, 39.5), turned to 180 degrees
- moved C15 213.1 mm to (156.0, 109.5), turned to 90 degrees
- moved C50 193.8 mm to (152.0, 57.5)
- moved D7 191.3 mm to (132.0, 46.5), turned to 180 degrees
- moved R17 182.8 mm to (153.5, 109.5), turned to 90 degrees
- moved R22 182.3 mm to (139.5, 68.5)
- moved R14 180.5 mm to (169.5, 106.0), turned to 270 degrees
- moved R19 180.2 mm to (162.0, 109.5), turned to 270 degrees
- moved R23 179.9 mm to (135.5, 46.5)
- moved C9 177.5 mm to (171.5, 106.0), turned to 270 degrees
- moved R20 175.0 mm to (174.5, 112.5)
- moved R18 174.7 mm to (167.0, 109.5), turned to 90 degrees
- moved C8 174.7 mm to (160.5, 100.5), turned to 180 degrees
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Connections:
- net Net-(Q7-Pad1) renamed /h-bridge/LO_1
- net Net-(Q9-Pad1) renamed /h-bridge/LO_2
- C2 pad 2: GNDA -> GND
- C20 pad 1: +3V3 -> +3V3A
- C4 pad 2: GNDA -> GND
- C48 pad 2: GNDA -> GND
- C49 pad 2: GNDA -> GND
- C5 pad 1: /mcu/BRIDGE_TEMP -> /mcu/I_SENSOR_OUT
- C5 pad 2: GNDA -> GND
- C60 pad 1: Net-(C60-Pad1) -> /h-bridge/VBOOT_1
- C60 pad 2: Net-(C60-Pad2) -> /h-bridge/HS_1
- C67 pad 1: Net-(C67-Pad1) -> /h-bridge/VBOOT_2
- C67 pad 2: Net-(C67-Pad2) -> /h-bridge/HS_2
- C72 pad 2: GND -> GNDA
- C74 pad 2: GNDA -> GND
- C76 pad 1: /mcu/BRIDGE_TEMP -> /mcu/MOTOR_TEMP
- C76 pad 2: GNDA -> GND
- C77 pad 1: /sensors/BRIDGE_TEMP -> /mcu/BRIDGE_TEMP
- C77 pad 2: GNDA -> GND
- D13 pad 1: Net-(C60-Pad2) -> /h-bridge/HS_1
- D14 pad 1: Net-(C67-Pad2) -> /h-bridge/HS_2
- P11 pad 1: /h-bridge/I_SENSE- -> /h-bridge/I_SENSE+
- P13 pad 1: GNDA -> GND
- P13 pad 2: /mcu/BRIDGE_TEMP -> /mcu/MOTOR_TEMP
- P14 pad 1: GNDA -> GND
- P14 pad 2: /sensors/BRIDGE_TEMP -> /mcu/BRIDGE_TEMP
- P5 pad 1: GND -> /mcu/MCU_UART_RX
- P5 pad 2: /mcu/MCU_UART_RX -> /mcu/MCU_UART_TX
- P5 pad 3: /mcu/MCU_UART_TX -> GND
- Q6 pad 1: Net-(Q6-Pad1) -> /h-bridge/HO_1
- Q6 pad 3: /h-bridge/I_SENSE+ -> /h-bridge/I_SENSE-
- Q7 pad 2: /h-bridge/I_SENSE+ -> /h-bridge/I_SENSE-
- Q8 pad 1: Net-(Q8-Pad1) -> /h-bridge/HO_2
- R3 pad 2: GNDA -> GND
- R33 pad 1: Net-(R33-Pad1) -> /mcu/JTAG_RST_N
- R33 pad 2: GND -> Net-(R33-Pad2)
- R37 pad 1: /h-bridge/VBUS_EN_GD -> GNDPWR
- R37 pad 2: GNDPWR -> Net-(Q10-Pad1)
- R38 pad 2: /mcu/BRIDGE_TEMP -> /mcu/MOTOR_TEMP
- R40 pad 1: /h-bridge/VBUS_DIS_GD -> GNDPWR
- R40 pad 2: GNDPWR -> Net-(Q3-Pad1)
- R41 pad 1: /h-bridge/VBUS_ST_GD -> Net-(Q4-Pad1)
- R47 pad 1: /h-bridge/I_SENSE+ -> /h-bridge/I_SENSE-
- R47 pad 2: Net-(C60-Pad2) -> /h-bridge/HS_1
- R48 pad 2: Net-(C67-Pad2) -> /h-bridge/HS_2
- R59 pad 2: /sensors/BRIDGE_TEMP -> /mcu/BRIDGE_TEMP
- R8 pad 1: /mcu/BRIDGE_TEMP -> /mcu/I_SENSOR_OUT
- RV1 pad 1: Net-(R4-Pad1) -> Net-(RV1-Pad1)
- RV1 pad 2: Net-(RV1-Pad2) -> Net-(R4-Pad1)
- SW2 pad 1: Net-(R33-Pad1) -> GND
- SW2 pad 2: /mcu/JTAG_RST_N -> Net-(R33-Pad2)
- U10 pad 4: +3V3 -> +3V3A
- U10 pad 6: +3V3 -> +3V3A
- U13 pad 1: /mcu/BRIDGE_TEMP -> /mcu/VBAT_CTRL
- U13 pad 10: GNDA -> GND
- U13 pad 107: Net-(U13-Pad107) -> /mcu/DEBUG_0
- U13 pad 108: Net-(U13-Pad108) -> /mcu/DEBUG_1
- U13 pad 109: Net-(U13-Pad109) -> /mcu/DEBUG_2
- U13 pad 110: Net-(U13-Pad110) -> /mcu/DEBUG_3
- U13 pad 116: Net-(U13-Pad116) -> /mcu/MCU_UART_RX
- U13 pad 117: Net-(U13-Pad117) -> /mcu/MCU_UART_TX
- U13 pad 12: /mcu/BRIDGE_TEMP -> Net-(U13-Pad12)
- U13 pad 125: Net-(U13-Pad125) -> /mcu/DEBUG_4
- U13 pad 126: Net-(U13-Pad126) -> /mcu/DEBUG_5
- U13 pad 127: Net-(U13-Pad127) -> /mcu/DEBUG_6
- U13 pad 128: Net-(U13-Pad128) -> /mcu/DEBUG_7
- U13 pad 15: /sensors/BRIDGE_TEMP -> Net-(U13-Pad15)
- U13 pad 19: /mcu/VBAT_CTRL -> /mcu/VBUS_MOTOR
- U13 pad 21: Net-(U13-Pad21) -> /mcu/I_SENSOR_OUT
- U13 pad 3: Net-(U13-Pad3) -> /mcu/BRIDGE_TEMP
- U13 pad 33: /mcu/DEBUG_0 -> Net-(U13-Pad33)
- U13 pad 34: /mcu/DEBUG_1 -> Net-(U13-Pad34)
- U13 pad 35: /mcu/DEBUG_2 -> Net-(U13-Pad35)
- U13 pad 36: /mcu/DEBUG_3 -> Net-(U13-Pad36)
- U13 pad 37: /mcu/DEBUG_4 -> Net-(U13-Pad37)
- U13 pad 38: /mcu/DEBUG_5 -> Net-(U13-Pad38)
- U13 pad 4: /mcu/VBUS_MOTOR -> /mcu/MOTOR_TEMP
- U13 pad 40: /mcu/DEBUG_6 -> /h-bridge/VBUS_EN_MCU
- U13 pad 41: /mcu/DEBUG_7 -> /h-bridge/VBUS_ST_MCU
- U13 pad 42: Net-(U13-Pad42) -> /h-bridge/VBUS_DIS_MCU
- U13 pad 5: Net-(JP1-Pad1) -> Net-(U13-Pad5)
- U13 pad 62: /mcu/PWM_FAN -> Net-(U13-Pad62)
- U13 pad 63: /h-bridge/VBUS_DIS_MCU -> Net-(U13-Pad63)
- U13 pad 71: /h-bridge/VBUS_EN_MCU -> Net-(U13-Pad71)
- U13 pad 72: /h-bridge/VBUS_ST_MCU -> Net-(U13-Pad72)
- U13 pad 74: Net-(U13-Pad74) -> Net-(JP1-Pad1)
- U13 pad 91: Net-(U13-Pad91) -> /mcu/PWM_FAN
- U16 pad 13: /h-bridge/VBUS_DIS_GD -> /h-bridge/VBUS_ST_GD
- U16 pad 14: /h-bridge/VBUS_ST_GD -> /h-bridge/VBUS_DIS_GD
- U16 pad 3: /h-bridge/VBUS_ST_MCU -> /h-bridge/VBUS_DIS_MCU
- U16 pad 4: /h-bridge/VBUS_DIS_MCU -> /h-bridge/VBUS_ST_MCU
- U19 pad 2: Net-(C60-Pad1) -> /h-bridge/VBOOT_2
- U19 pad 3: Net-(Q6-Pad1) -> /h-bridge/HO_2
- U19 pad 4: Net-(C60-Pad2) -> /h-bridge/HS_2
- U19 pad 5: Net-(R44-Pad1) -> /h-bridge/PWM3_GD
- U19 pad 6: Net-(R45-Pad1) -> /h-bridge/PWM4_GD
- U19 pad 7: /h-bridge/PWM1_GD -> GNDPWR
- U19 pad 8: /h-bridge/PWM2_GD -> Net-(R49-Pad2)
- U20 pad 11: /h-bridge/PWM4_GD -> /h-bridge/PWM2_GD
- U20 pad 12: /h-bridge/PWM3_GD -> /h-bridge/PWM1_GD
- U20 pad 13: /h-bridge/PWM2_GD -> /h-bridge/PWM4_GD
- U20 pad 14: /h-bridge/PWM1_GD -> /h-bridge/PWM3_GD
- U20 pad 3: /h-bridge/PWM1_MCU -> /h-bridge/PWM3_MCU
- U20 pad 4: /h-bridge/PWM2_MCU -> /h-bridge/PWM4_MCU
- U20 pad 5: /h-bridge/PWM3_MCU -> /h-bridge/PWM1_MCU
- U20 pad 6: /h-bridge/PWM4_MCU -> /h-bridge/PWM2_MCU
- U3 pad 5: GNDA -> GND
- U4 pad 2: GNDA -> GND
- U4 pad 3: GNDA -> GND
- U5 pad 2: GNDA -> GND
Routing:
- net +12V_ISO: track 8.53 -> 79.3 mm, vias 0 -> 4
- net /h-bridge/PWM2_GD: track 0.00 -> 54.0 mm, vias 0 -> 2
- net /h-bridge/I_SENSE-: track 27.8 -> 77.5 mm, vias 0 -> 5
- net /h-bridge/PWM1_GD: track 0.00 -> 49.7 mm, vias 0 -> 2
- net /h-bridge/I_SENSE+: track 71.6 -> 27.8 mm
- net /h-bridge/PWM3_GD: track 0.00 -> 27.4 mm, vias 0 -> 2
- net /h-bridge/PWM4_GD: track 0.00 -> 25.1 mm, vias 0 -> 2
- net /h-bridge/PWM1_MCU: track 0.00 -> 22.9 mm
- net /mcu/VBUS_MOTOR: track 0.00 -> 20.2 mm
- net Net-(C67-Pad2): track 19.1 -> 0.00 mm, vias 2 -> 0
- net /h-bridge/VBUS_DIS_MCU: track 0.00 -> 15.4 mm
- net /h-bridge/VBUS_EN_MCU: track 0.00 -> 15.3 mm
- net /h-bridge/VBUS_ST_MCU: track 0.00 -> 15.2 mm
- net /h-bridge/HO_2: track 0.00 -> 13.3 mm, vias 0 -> 6
- net /h-bridge/PWM4_MCU: track 0.00 -> 13.3 mm
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- added copper zone on F.Cu, net +12V_ISO
- added copper zone on B.Cu, net /h-bridge/HO_1
- added copper zone on F.Cu, net /h-bridge/HO_1
- added copper zone on B.Cu, net /h-bridge/HO_2
- added copper zone on F.Cu, net /h-bridge/HO_2
- added copper zone on F.Cu, net /h-bridge/HS_1
- added copper zone on F.Cu, net /h-bridge/HS_2
- added copper zone on In2.Cu, net /h-bridge/I_SENSE-
- added copper zone on In2.Cu, net /h-bridge/LO_1
- added copper zone on F.Cu, net /h-bridge/LO_2
- added copper zone on In2.Cu, net /h-bridge/LO_2
- added copper zone on F.Cu, net /h-bridge/M-
- added copper zone on In2.Cu, net /h-bridge/M-
- added copper zone on F.Cu, net /h-bridge/VBOOT_1
- added copper zone on F.Cu, net /h-bridge/VBOOT_2
- added copper zone on In1.Cu, net GND
- added copper zone on F.Cu, net GNDPWR
- added copper zone on F.Cu, net Net-(R46-Pad2)
- added copper zone on F.Cu, net Net-(R49-Pad2)
Other:
- board size 170 x 88 mm -> 180 x 88 mm
- net class Default: clearance 0.2 -> 0.1524
- rule trace_clearance: 0.2 -> 0.1524
- rule trace_min: 0.2 -> 0.1524
- board text added: "+12 OK"
- board text added: "-12 OK"
- board text added: "0603 max = 0.1W consider going to 0805"
- board text added: "1 2 3 4"
- board text added: "1 JTAG 9"
- board text added: "12V ISO OK"
- board text added: "3V3 OK"
- board text added: "D0 D1 D2 D3 D4 D5 D6 D7"
- board text added: "FACTORY RESET"
- board text added: "RESET"
- board text added: "STATUS"
- board text added: "TX RX GND"
- board text added: "UART"

Commit message: more layout progress
Parts:
- removed D1: MBRM-120, 2kwMotorController:DIODE_POWERMITE
- removed FB1: FERRITE_BEAD, Capacitors_SMD:C_0603
- C10: value 100n -> 10u; moved to B.Cu
- C12: moved to B.Cu
- C72: value 1u -> 10u; footprint Capacitors_SMD:C_0603 -> Capacitors_SMD:C_0805
- R56: value 2.2 -> 1
- U14: footprint 2kwMotorController:VSSOP8 -> Housings_SSOP:MSOP-8_3x3mm_Pitch0.65mm
- U19, U6: footprint Housings_SOIC:SOIC-8-1EP_3.9x4.9mm_Pitch1.27mm -> 2kwMotorController:SOIC-8-1EP_3.9x4.9mm_Pitch1.27mm
- U9: value LF33ABDT -> R-78E3.3-0.5; footprint TO_SOT_Packages_SMD:TO-252-2Lead -> 2kwMotorController:R-78E-0.5; moved to B.Cu
- moved P3 65.5 mm to (192.5, 46.0)
- moved R15 22.5 mm to (209.5, 71.0)
- moved C17 21.9 mm to (152.0, 95.2)
- moved D4 21.8 mm to (209.5, 68.0)
- moved C21 20.9 mm to (173.2, 102.8), turned to 90 degrees
- moved C19 18.8 mm to (154.2, 95.5)
- moved R12 18.0 mm to (199.0, 67.0), turned to 270 degrees
- moved D3 16.7 mm to (152.8, 106.2)
- moved C12 16.0 mm to (203.5, 59.5), turned to 0 degrees
- moved L3 16.0 mm to (153.0, 101.5)
- moved C18 15.9 mm to (171.2, 102.8), turned to 90 degrees
- moved Q1 15.3 mm to (203.0, 69.5)
- moved D6 13.9 mm to (168.0, 119.5)
- moved R21 13.7 mm to (171.2, 119.5)
- moved D2 13.3 mm to (168.2, 104.2), turned to 180 degrees
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Connections:
- net Net-(C9-Pad1) renamed /power/SMPS_SHDN
- C13 pad 2: Net-(C13-Pad2) -> /power/SMPS_SW2
- C14 pad 2: Net-(C14-Pad2) -> /power/SMPS_VREF
- C15 pad 2: Net-(C15-Pad2) -> /power/SMPS_FB1N
- C16 pad 2: Net-(C16-Pad2) -> /power/SMPS_FB2P
- C20 pad 2: GNDA -> GND
- C22 pad 2: GNDA -> GND
- C72 pad 1: Net-(C72-Pad1) -> +3V3A
- C72 pad 2: GNDA -> GND
- D2 pad 2: Net-(D2-Pad2) -> /power/SMPS_SW1
- L1 pad 2: Net-(D2-Pad2) -> /power/SMPS_SW1
- L2 pad 2: Net-(C13-Pad2) -> /power/SMPS_SW2
- P1 pad 1: +BATT -> GNDCBAT
- P1 pad 2: GNDCBAT -> +BATT
- R16 pad 2: Net-(C15-Pad2) -> /power/SMPS_FB1N
- R17 pad 2: Net-(C15-Pad2) -> /power/SMPS_FB1N
- R18 pad 1: Net-(C14-Pad2) -> /power/SMPS_VREF
- R18 pad 2: Net-(C16-Pad2) -> /power/SMPS_FB2P
- R19 pad 1: Net-(C16-Pad2) -> /power/SMPS_FB2P
- R56 pad 1: Net-(C72-Pad1) -> +3V3
- U10 pad 2: GNDA -> GND
- U10 pad 3: GNDA -> GND
- U10 pad 5: GNDA -> GND
- U8 pad 1: Net-(C15-Pad2) -> GND
- U8 pad 10: Net-(D2-Pad2) -> /power/SMPS_SW2
- U8 pad 2: Net-(C14-Pad2) -> /power/SMPS_FB2P
- U8 pad 3: Net-(C14-Pad2) -> /power/SMPS_VREF
- U8 pad 4: Net-(C16-Pad2) -> /power/SMPS_VREF
- U8 pad 5: GND -> /power/SMPS_FB1N
- U8 pad 6: Net-(C13-Pad2) -> /power/SMPS_SW1
Routing:
- net +BATT: track 0.00 -> 92.8 mm, vias 0 -> 2
- net +12V: track 0.00 -> 83.5 mm
- net +5V: track 0.00 -> 29.9 mm
- net Net-(D8-Pad2): track 0.00 -> 22.7 mm
- net -12V: track 0.00 -> 19.8 mm
- net GND: track 0.00 -> 19.3 mm, vias 0 -> 15
- net +3V3: track 4.56 -> 21.9 mm
- net /power/SMPS_SHDN: track 0.00 -> 12.6 mm, vias 0 -> 3
- net Net-(Q2-Pad4): track 0.00 -> 9.16 mm
- net /power/SMPS_FB2P: track 0.00 -> 9.07 mm
- net /power/SMPS_FB1N: track 0.00 -> 8.65 mm
- net /mcu/ENCODER_CHB: track 0.00 -> 8.05 mm
- net /mcu/ENCODER_CHA: track 0.00 -> 7.85 mm
- net (no net): track 0.00 -> 6.97 mm
- net /power/SMPS_VREF: track 0.00 -> 5.36 mm
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- added copper zone on F.Cu, net +12V
- added copper zone on In2.Cu, net +12V
- added copper zone on In2.Cu, net +3V3A
- added copper zone on B.Cu, net +BATT
- added copper zone on In2.Cu, net -12V
- added copper zone on F.Cu, net /power/SMPS_SW1
- added copper zone on F.Cu, net /power/SMPS_SW2
- added copper zone on F.Cu, net GND
Other:
- net class Default: via_drill 0.4 -> 0.3
- rule via_min_drill: 0.300025 -> 0.3
- rule via_min_size: 0.450012 -> 0.6
- board text added: "+BATT"
- board text added: "-FAN+"
- board text added: "BRIDGE TEMP SENSOR"
- board text added: "GND IDX CA 5V CB"
- board text added: "GND V+"
- board text added: "MOTOR TEMP SENSOR"
- board text added: "RX TX GND"
- board text removed: "+12 OK"
- board text removed: "+FAN-"
- board text removed: "-12 OK"
- board text removed: "0603 max = 0.1W consider going to 0805"
- board text removed: "1 2 3 4"
- board text removed: "1 JTAG 9"
- board text removed: "12V ISO OK"
- board text removed: "2kW DC MOTOR CONTROLLER OFD 2017"
- board text removed: "3V3 OK"
- board text removed: "BRIDGE TEMP PROBE"
- board text removed: "FACTORY RESET"
- board text removed: "GND IDX A 5V B"
- board text removed: "MOTOR TEMP PROBE"
- board text removed: "RESET"
- board text removed: "STATUS"
- board text removed: "TX RX GND"
- board text removed: "V+"
- board text removed: "V+ GND"
- board text removed: "V-"
- board text removed: "VBUS"

Commit message: All routing finished
Parts:
- added R44: 18k, Resistors_SMD:R_0603, F.Cu at (137.5, 33.0)
- added R45: 2k, Resistors_SMD:R_0603, F.Cu at (140.4, 31.4)
- C1, C3: value 47p -> 10p
- C32, C33, C37, C38, C40, C42, C43, C44: moved to B.Cu
- C4: value 47n -> 100n
- P3: value CONN_01X08_DEBUG -> CONN_01X09; footprint Pin_Headers:Pin_Header_Straight_1x08 -> Pin_Headers:Pin_Header_Straight_1x09
- R1: value 1.2M -> 120k
- R7: value 100 -> 47
- U1: value LM358 -> LM358A; footprint SMD_Packages:SOIC-8-N -> Housings_SOIC:SOIC-8_3.9x4.9mm_Pitch1.27mm
- moved C37 155.7 mm to (172.5, 66.8), turned to 180 degrees
- moved C36 149.9 mm to (182.5, 65.8)
- moved C41 149.9 mm to (169.0, 73.2), turned to 270 degrees
- moved C44 149.8 mm to (176.0, 67.5)
- moved R58 149.6 mm to (179.0, 82.8), turned to 90 degrees
- moved C43 148.8 mm to (172.5, 65.0), turned to 180 degrees
- moved R57 148.7 mm to (175.8, 82.8), turned to 270 degrees
- moved C49 148.5 mm to (175.8, 49.0)
- moved C45 148.4 mm to (164.5, 51.8), turned to 180 degrees
- moved C48 146.5 mm to (175.8, 50.5)
- moved C32 145.7 mm to (167.6, 66.9)
- moved C33 144.6 mm to (167.5, 56.8)
- moved C35 143.9 mm to (161.0, 56.5), turned to 90 degrees
- moved C40 141.5 mm to (175.5, 60.8), turned to 180 degrees
- moved C38 141.4 mm to (165.9, 62.6), turned to 90 degrees
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Connections:
- net Net-(C34-Pad1) renamed /mcu/VDDC
- P6 pad 1: /mcu/CANH -> /mcu/CANL
- P6 pad 2: /mcu/CANL -> /mcu/CANH
- R1 pad 2: /h-bridge/VBUS -> Net-(R1-Pad2)
- U1 pad 1: Net-(C1-Pad1) -> Net-(R1-Pad2)
- U1 pad 2: Net-(C1-Pad2) -> Net-(R1-Pad2)
- U1 pad 3: GND -> Net-(R44-Pad2)
- U1 pad 5: (no net) -> GNDPWR
- U1 pad 6: (no net) -> Net-(C1-Pad2)
- U1 pad 7: (no net) -> Net-(C1-Pad1)
- U13 pad 103: Net-(U13-Pad103) -> /mcu/LED_0
- U13 pad 104: Net-(U13-Pad104) -> /mcu/LED_1
- U13 pad 105: Net-(U13-Pad105) -> /mcu/LED_2
- U13 pad 106: Net-(U13-Pad106) -> /mcu/LED_3
- U13 pad 22: /mcu/LED_3 -> Net-(U13-Pad22)
- U13 pad 23: /mcu/LED_2 -> Net-(U13-Pad23)
- U13 pad 24: /mcu/LED_1 -> Net-(U13-Pad24)
- U13 pad 25: /mcu/LED_0 -> Net-(U13-Pad25)
- U13 pad 3: /mcu/BRIDGE_TEMP -> /mcu/MOTOR_TEMP
- U13 pad 4: /mcu/MOTOR_TEMP -> /mcu/BRIDGE_TEMP
Routing:
- net +12V_ISO: track 79.3 -> 241.4 mm, vias 4 -> 9
- net /h-bridge/VBUS_ST_GD: track 0.00 -> 132.9 mm, vias 0 -> 4
- net /h-bridge/VBUS_DIS_GD: track 0.16 -> 124.3 mm, vias 0 -> 2
- net GND: track 19.3 -> 126.5 mm, vias 15 -> 59
- net /h-bridge/VBUS_EN_GD: track 0.00 -> 86.1 mm, vias 0 -> 3
- net /h-bridge/PWM3_GD: track 27.4 -> 110.9 mm
- net /h-bridge/PWM4_GD: track 25.1 -> 102.7 mm
- net +BATT: track 92.8 -> 147.5 mm, vias 2 -> 3
- net +3V3: track 21.9 -> 72.0 mm, vias 0 -> 15
- net /mcu/QEI_PHB: track 0.00 -> 42.5 mm, vias 0 -> 2
- net /mcu/QEI_PHA: track 0.00 -> 42.3 mm, vias 0 -> 2
- net /mcu/PWM_FAN: track 0.00 -> 42.3 mm, vias 0 -> 4
- net /mcu/BRIDGE_TEMP: track 2.31 -> 41.9 mm
- net /mcu/DEBUG_0: track 0.00 -> 38.9 mm
- net Net-(C2-Pad1): track 0.00 -> 36.6 mm, vias 0 -> 1
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- added copper zone on In2.Cu, net +3V3
- added copper zone on F.Cu, net +BATT
- added copper zone on B.Cu, net GND
Other:
- board text added: "+3V3 OK"
- board text added: "0 STATUS 3"
- board text added: "CANL CANH GND"
- board text added: "FACTORY RESET"
- board text added: "GND D7 D6 D5 D4 D3 D2 D1 D0"
- board text added: "ID0 ID1"
- board text added: "RESET"
- board text removed: "CANH CANL GND"
- board text removed: "D0 D1 D2 D3 D4 D5 D6 D7"

Commit message: layout cleanup, add buffer for fan drive
Parts:
- added C82: 100n, Capacitors_SMD:C_0603, F.Cu at (190.4, 107.2)
- added REF**111: VIA-0.6mm, 2kwMotorController:VIA-0.6mm, F.Cu at (152.5, 96.8)
- added REF**111: VIA-0.6mm, 2kwMotorController:VIA-0.6mm, F.Cu at (156.0, 109.5)
- added REF**111: VIA-0.6mm, 2kwMotorController:VIA-0.6mm, F.Cu at (170.6, 102.8)
- added REF**111: VIA-0.6mm, 2kwMotorController:VIA-0.6mm, F.Cu at (194.6, 107.1)
- added REF**111: VIA-0.6mm, 2kwMotorController:VIA-0.6mm, F.Cu at (184.8, 110.1)
- added REF**1111: VIA-0.6mm, 2kwMotorController:VIA-0.6mm, F.Cu at (193.2, 109.0)
- added REF**11111: VIA-0.6mm, 2kwMotorController:VIA-0.6mm, F.Cu at (169.2, 106.5)
- added REF**11111: VIA-0.6mm, 2kwMotorController:VIA-0.6mm, F.Cu at (169.2, 107.0)
- added REF**11111: VIA-0.6mm, 2kwMotorController:VIA-0.6mm, F.Cu at (159.1, 105.2)
- added REF**11111: VIA-0.6mm, 2kwMotorController:VIA-0.6mm, F.Cu at (159.1, 105.7)
- added REF**11112: VIA-0.6mm, 2kwMotorController:VIA-0.6mm, F.Cu at (169.2, 107.5)
- added REF**11112: VIA-0.6mm, 2kwMotorController:VIA-0.6mm, F.Cu at (159.1, 106.1)
- added REF**11113: VIA-0.6mm, 2kwMotorController:VIA-0.6mm, F.Cu at (159.1, 106.7)
- added REF**11114: VIA-0.6mm, 2kwMotorController:VIA-0.6mm, F.Cu at (159.1, 107.2)
- added REF**1112: VIA-0.6mm, 2kwMotorController:VIA-0.6mm, F.Cu at (193.2, 109.5)
- added REF**11121: VIA-0.6mm, 2kwMotorController:VIA-0.6mm, F.Cu at (169.8, 106.5)
- added REF**11121 (x2): VIA-0.6mm, 2kwMotorController:VIA-0.6mm, F.Cu at (169.8, 107.0)
- added REF**11122 (x2): VIA-0.6mm, 2kwMotorController:VIA-0.6mm, F.Cu at (169.8, 107.5)
- added REF**1113: VIA-0.6mm, 2kwMotorController:VIA-0.6mm, F.Cu at (193.2, 110.0)
- added REF**112: VIA-0.6mm, 2kwMotorController:VIA-0.6mm, F.Cu at (184.8, 110.6)
- added REF**112: VIA-0.6mm, 2kwMotorController:VIA-0.6mm, F.Cu at (156.0, 110.0)
- added REF**112: VIA-0.6mm, 2kwMotorController:VIA-0.6mm, F.Cu at (152.5, 97.2)
- added REF**113: VIA-0.6mm, 2kwMotorController:VIA-0.6mm, F.Cu at (184.8, 111.1)
- added REF**113: VIA-0.6mm, 2kwMotorController:VIA-0.6mm, F.Cu at (156.0, 110.5)
- added REF**114: VIA-0.6mm, 2kwMotorController:VIA-0.6mm, F.Cu at (184.8, 111.6)
- added REF**114: VIA-0.6mm, 2kwMotorController:VIA-0.6mm, F.Cu at (156.0, 111.0)
- added REF**115: VIA-0.6mm, 2kwMotorController:VIA-0.6mm, F.Cu at (184.8, 112.1)
- added REF**115: VIA-0.6mm, 2kwMotorController:VIA-0.6mm, F.Cu at (156.0, 111.5)
- added REF**116: VIA-0.6mm, 2kwMotorController:VIA-0.6mm, F.Cu at (184.8, 112.6)
- added REF**121: VIA-0.6mm, 2kwMotorController:VIA-0.6mm, F.Cu at (195.1, 107.1)
- added REF**121: VIA-0.6mm, 2kwMotorController:VIA-0.6mm, F.Cu at (171.1, 102.8)
- added REF**121: VIA-0.6mm, 2kwMotorController:VIA-0.6mm, F.Cu at (153.0, 96.8)
- added REF**122: VIA-0.6mm, 2kwMotorController:VIA-0.6mm, F.Cu at (153.0, 97.2)
- added REF**131: VIA-0.6mm, 2kwMotorController:VIA-0.6mm, F.Cu at (195.6, 107.1)
- added REF**131: VIA-0.6mm, 2kwMotorController:VIA-0.6mm, F.Cu at (171.6, 102.8)
- added REF**131: VIA-0.6mm, 2kwMotorController:VIA-0.6mm, F.Cu at (153.5, 96.8)
- added REF**132: VIA-0.6mm, 2kwMotorController:VIA-0.6mm, F.Cu at (153.5, 97.2)
- added REF**141: VIA-0.6mm, 2kwMotorController:VIA-0.6mm, F.Cu at (196.1, 107.1)
- added REF**141: VIA-0.6mm, 2kwMotorController:VIA-0.6mm, F.Cu at (172.1, 102.8)
- added REF**141: VIA-0.6mm, 2kwMotorController:VIA-0.6mm, F.Cu at (154.0, 96.8)
- added REF**142: VIA-0.6mm, 2kwMotorController:VIA-0.6mm, F.Cu at (154.0, 97.2)
- added REF**151: VIA-0.6mm, 2kwMotorController:VIA-0.6mm, F.Cu at (196.6, 107.1)
- added REF**151: VIA-0.6mm, 2kwMotorController:VIA-0.6mm, F.Cu at (172.6, 102.8)
- added REF**161: VIA-0.6mm, 2kwMotorController:VIA-0.6mm, F.Cu at (197.1, 107.1)
- added REF**161: VIA-0.6mm, 2kwMotorController:VIA-0.6mm, F.Cu at (173.1, 102.8)
- added U21: 74LVC1G17, 2kwMotorController:SC-74A, F.Cu at (186.4, 105.0)
- R24: value 100 -> 180
- moved R25 8.19 mm to (186.4, 100.4), turned to 270 degrees
- moved R20 8.02 mm to (174.0, 111.8), turned to 90 degrees
- moved D5 6.77 mm to (172.0, 111.8), turned to 90 degrees
- moved D6 6.77 mm to (179.0, 111.8), turned to 90 degrees
- moved D3 4.05 mm to (156.8, 106.2), turned to 180 degrees
- moved R31 2.46 mm to (196.2, 84.0)
- moved D2 2.21 mm to (167.2, 106.2), turned to 90 degrees
- moved C18 2.02 mm to (171.0, 104.8)
- moved C21 2.02 mm to (173.0, 104.8)
- moved R21 1.58 mm to (177.0, 111.8), turned to 90 degrees
- moved C17 1.12 mm to (152.5, 94.2)
- moved R17 0.90 mm to (165.2, 110.6)
- moved C19 0.79 mm to (155.0, 95.2), turned to 180 degrees
- moved R16 0.70 mm to (167.8, 111.3)
- moved D8 0.61 mm to (196.2, 112.2), turned to 180 degrees
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Connections:
- R24 pad 2: /mcu/PWM_FAN -> Net-(R24-Pad2)
- R25 pad 2: Net-(Q2-Pad4) -> /mcu/PWM_FAN
Routing:
- net -12V: track 19.8 -> 59.5 mm, vias 0 -> 2
- net GND: track 126.5 -> 147.6 mm, vias 59 -> 72
- net +5V: track 29.9 -> 44.7 mm
- net Net-(D8-Pad2): track 22.7 -> 12.8 mm
- net /power/SMPS_FB1N: track 8.65 -> 3.42 mm
- net /mcu/PWM_FAN: track 42.3 -> 39.1 mm
- net +12V: track 86.2 -> 83.9 mm
- net Net-(D6-Pad1): track 0.00 -> 2.00 mm
- net Net-(D5-Pad1): track 0.00 -> 2.00 mm
- net Net-(R24-Pad2): track 0.00 -> 1.80 mm
- net /power/SMPS_SW1: track 2.00 -> 0.30 mm, vias 1 -> 0
- net Net-(Q2-Pad4): track 9.16 -> 7.75 mm
- net Net-(R31-Pad1): track 2.12 -> 2.75 mm
- added copper zone on F.Cu, net -12V
- added copper zone on F.Cu, net Net-(C13-Pad1)
- added copper zone on F.Cu, net Net-(D8-Pad2)
Other:
- board text added: "+12V -12V"
- board text added: "+3V3"
- board text removed: "+3V3 OK"
