File: hardware/2kwMotorController.kicad_pcb (KiCad board)
At the start: 4 copper layers, 182 x 88 mm, 410 parts, among them M1 MOUNTING_HOLE, M2 MOUNTING_HOLE, M3 MOUNTING_HOLE, M4 MOUNTING_HOLE, M5 MOUNTING_HOLE, M6 MOUNTING_HOLE, P1 CONN_01X02_CBAT, P10 CONN_01_BRK, P11 CONN_01_M+, P12 CONN_01_M-, P13 CONN_01X02_MTMP, P14 CONN_01X02_BTMP, P2 CONN_01X02_FAN, P3 CONN_01X09, P4 CONN_02X05_JTAG, P5 CONN_01X03_UART, P6 CONN_01X03_CAN, P7 CONN_01X05_ENCODER, P8 CONN_01_V+, P9 CONN_01_V-, Q1 DMG4712SSS, Q10 PSMN021-100, Q2 DMG4712SSS, Q3 IRFP4468, Q4 PSMN021-100, Q5 IRFP4468, Q6 IRFP4468, Q7 IRFP4468, Q8 IRFP4468, Q9 IRFP4468, SW2 SW_PUSH, U1 LM358A, U10 MCP1501T-30E, U11 PDM1-S, U12 MIC5225-5.0, U13 TM4C1294KCPDT, U14 74LVCH2T45, U15 SN65HVD231D, U16 Si8045AA, U17 MIC4127, U18 MIC4127, U19 UCC27211, U2 LAH-100P, U20 Si8045AA, U21 74LVC1G17, U3 LOC110, U4 MCP6001, U5 ADA4805-1, U6 UCC27211, U7 MIC5225-5.0, U8 LT3471, U9 R-78E3.3-0.5, Y1 NX5032GA

Commit message: Revised layout mostly complete
Parts:
- removed D10, D11, D12, D9: LED, LEDs:LED_0603
- removed the GND at (153.5, 113.5)
- removed GND_ISO (x4): GND_POINT, Pin_Headers:Pin_Header_Straight_1x01
- removed M1, M2, M4, M5: MOUNTING_HOLE, 2kwMotorController:M4-SCREW-HOLE
- removed R30: 120, Resistors_SMD:R_0603
- removed R65: 150, 2kwMotorController:RESISTOR_FMP200
- added C83: 560u, 2kwMotorController:CP18, F.Cu at (70.0, 28.0)
- added C84: 560u, 2kwMotorController:CP18, F.Cu at (125.0, 28.0)
- added C85: 100n, Capacitors_SMD:C_0603, F.Cu at (167.2, 85.0)
- added C86: 100n, Capacitors_SMD:C_0603, F.Cu at (167.2, 88.5)
- added GND1, GND2, GND8, GND9: GND_POINT, Pin_Headers:Pin_Header_Straight_1x01, F.Cu at (118.5, 126.1)
- added JP2: Jumper_NO_Small, Pin_Headers:Pin_Header_Straight_1x02, F.Cu at (192.0, 69.0)
- added P15: CONN_01X04, Pin_Headers:Pin_Header_Straight_1x04, F.Cu at (199.0, 51.5)
- added REF**: M4-SCREW-HOLE, 2kwMotorController:M4-SCREW-HOLE, F.Cu at (57.0, 93.5)
- added REF**: M4-SCREW-HOLE, 2kwMotorController:M4-SCREW-HOLE, F.Cu at (87.5, 93.5)
- added REF**: M4-SCREW-HOLE, 2kwMotorController:M4-SCREW-HOLE, F.Cu at (118.0, 93.5)
- added REF**: M3-SCREW-HOLE, 2kwMotorController:M3-SCREW-HOLE, F.Cu at (199.0, 28.5)
- added REF**: M3-SCREW-HOLE, 2kwMotorController:M3-SCREW-HOLE, F.Cu at (199.0, 57.5)
- added REF**: M3-SCREW-HOLE, 2kwMotorController:M3-SCREW-HOLE, F.Cu at (199.0, 97.5)
- added REF**: M4-SCREW-HOLE, 2kwMotorController:M4-SCREW-HOLE, F.Cu at (87.5, 44.5)
- added REF**: M4-SCREW-HOLE, 2kwMotorController:M4-SCREW-HOLE, F.Cu at (118.0, 44.5)
- added REF**: M4-SCREW-HOLE, 2kwMotorController:M4-SCREW-HOLE, F.Cu at (57.0, 44.5)
- added TP40: TEST_POINT, 2kwMotorController:TEST_PAD_1.27mm, F.Cu at (118.5, 126.1)
- added U22: SN74LVCH2T45, Housings_SSOP:MSOP-8_3x3mm_Pitch0.65mm, F.Cu at (164.2, 86.8)
- C10: footprint Capacitors_SMD:C_0603 -> Capacitors_SMD:C_0805
- C51, C52: value 1m -> 560u; footprint 2kwMotorController:Cap_Horizontal_D18_L36 -> 2kwMotorController:CP18
- P1: value CONN_01X02_CBAT -> CONN_01X02; footprint 2kwMotorController:TERM_2P_2-5_1990009 -> Pin_Headers:Pin_Header_Straight_1x02
- P13: value CONN_01X02_MTMP -> CONN_01X02; footprint 2kwMotorController:TERM_2P_2-5_1990009 -> Pin_Headers:Pin_Header_Straight_1x02
- P14: value CONN_01X02_BTMP -> CONN_01X02; footprint 2kwMotorController:TERM_2P_2-5_1990009 -> Pin_Headers:Pin_Header_Straight_1x02
- P2: value CONN_01X02_FAN -> CONN_01X04; footprint 2kwMotorController:TERM_2P_2-5_1990009 -> 2kwMotorController:TERM_4P_2-4_1990025
- P4: value CONN_02X05_JTAG -> CONN_02X05
- P6: value CONN_01X03_CAN -> CONN_01X03; footprint 2kwMotorController:TERM_3P_2-5_1990012 -> Pin_Headers:Pin_Header_Straight_1x03
- P7: value CONN_01X05_ENCODER -> CONN_01X05; footprint 2kwMotorController:TERM_5P_2-5_1990038 -> Pin_Headers:Pin_Header_Straight_1x05
- Q10, Q4: footprint 2kwMotorController:SOT-669_LFPAK_PASTE -> 2kwMotorController:SOT-669_LFPAK_ThermalVias-1
- R3: value 59.0 -> 59.0 0.1%
- R39: value 100 -> 10k
- U11: value PDM1-S -> PDM1-S12-S3
- U14: value 74LVCH2T45 -> SN74LVCH2T45
- moved R39 141.0 mm to (196.0, 95.0), turned to 90 degrees
- moved R33 101.6 mm to (186.8, -23.0)
- moved C52 77.0 mm to (105.0, 28.0), turned to 270 degrees
- moved SW2 59.7 mm to (189.0, 30.0), turned to 0 degrees
- moved R38 56.2 mm to (152.0, 0.50)
- moved GND 51.4 mm to (128.2, 6.50)
- moved JP1 51.2 mm to (190.0, 38.5), turned to 270 degrees
- moved TP7 49.5 mm to (156.2, 2.00)
- moved R57 45.4 mm to (219.0, 96.5)
- moved R58 45.4 mm to (222.2, 96.5)
- moved C77 44.2 mm to (155.0, 4.75)
- moved R59 43.6 mm to (158.2, 4.75)
- moved C76 42.4 mm to (155.5, 15.0)
- moved TP8 39.7 mm to (159.8, 1.75)
- moved REF**11 37.1 mm to (222.7, 51.4), turned to 90 degrees
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Connections:
- net /mcu/CAN_RX renamed /mcu/CAN1_RX
- net /mcu/CAN_TX renamed /mcu/CAN1_TX
- net /mcu/MCU_UART_RX renamed /mcu/MCU_UART3_RX
- net /mcu/MCU_UART_TX renamed /mcu/MCU_UART3_TX
- C52 pad 1: Net-(C52-Pad1) -> /h-bridge/VBUS
- C52 pad 2: /h-bridge/VBUS -> Net-(C51-Pad2)
- Q4 pad 2: Net-(C52-Pad1) -> Net-(C83-Pad2)
- R27 pad 1: GND -> /mcu/RED
- R27 pad 2: Net-(D9-Pad1) -> /mcu/LED_0
- R28 pad 1: GND -> /mcu/GREEN
- R28 pad 2: Net-(D10-Pad1) -> /mcu/LED_1
- R29 pad 1: GND -> /mcu/BLUE
- R29 pad 2: Net-(D11-Pad1) -> /mcu/LED_2
- R32 pad 1: /mcu/CANH -> Net-(JP2-Pad1)
- R32 pad 2: /mcu/CANL -> /mcu/CANH
- R39 pad 1: Net-(R39-Pad1) -> /mcu/ENCODER_INDEX
- R39 pad 2: /h-bridge/VBUS_ST_GATE_2 -> +5V
- U13 pad 106: /mcu/LED_3 -> Net-(U13-Pad106)
- U17 pad 4: /h-bridge/VBUS_ST_GD -> GNDPWR
- U17 pad 5: Net-(R39-Pad1) -> Net-(U17-Pad5)
Routing:
- net +BATT: track 146.0 -> 29.6 mm, vias 2 -> 0
- net /h-bridge/VBUS_ST_GD: track 132.3 -> 73.7 mm, vias 4 -> 3
- net Net-(C51-Pad2): track 22.6 -> 74.2 mm
- net +5V: track 52.0 -> 6.53 mm, vias 1 -> 0
- net /mcu/BRIDGE_TEMP: track 45.0 -> 0.00 mm
- net GND: track 185.1 -> 144.0 mm, vias 79 -> 57
- net /mcu/MOTOR_TEMP: track 37.9 -> 0.00 mm
- net /mcu/PWM_FAN: track 39.4 -> 2.36 mm, vias 2 -> 0
- net /mcu/JTAG_RST_N: track 39.7 -> 5.00 mm, vias 4 -> 0
- net /mcu/QEI_PHA: track 33.5 -> 0.11 mm, vias 2 -> 0
- net /mcu/CAN1_RX: track 33.1 -> 0.00 mm
- net /mcu/QEI_PHB: track 33.0 -> 0.00 mm, vias 2 -> 0
- net +12V_ISO: track 289.0 -> 260.3 mm, vias 4 -> 3
- net Net-(C52-Pad1): track 26.5 -> 0.00 mm
- net (no net): track 0.00 -> 25.7 mm, vias 0 -> 7
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- removed copper zone on F.Cu, net /power/FAN_DRAIN
- removed copper zone on In2.Cu, net /power/FAN_DRAIN
Other:
- board size 182 x 88 mm -> 170 x 97.8 mm
- board text added: "12V DC FAN + - + -"
- board text added: "2kw DC Motor Controller REV 1"
- board text added: "CANL CANH GND"
- board text added: "GND IDX A +5 B"
- board text added: "HBR TEMP"
- board text added: "MTR TEMP"
- board text added: "PWR IN GND 6-9V"
- board text added: "R G B GND"
- board text removed: "+ FAN - 12V DC"
- board text removed: "+3V3"
- board text removed: "- +"
- board text removed: "2kw DC Motor Controller REV 0"
- board text removed: "6V MIN 9V MAX"
- board text removed: "BRIDGE TEMP SENSOR"
- board text removed: "CANL GND CANH"
- board text removed: "GND CHA CHB INDEX +5V"
- board text removed: "GND VCC POWER IN"
- board text removed: "MOTOR TEMP SENSOR"
- board text removed: "STATUS S0 S1 S2 S3"

Commit message: Rev 1 layout finished
Parts:
- removed Q4: PSMN021-100, 2kwMotorController:SOT-669_LFPAK_ThermalVias-1
- removed R41: 10k, Resistors_SMD:R_0603
- removed R57, R58: 2.2k, Resistors_SMD:R_0603
- removed the REF**11 at (217.7, 52.0)
- removed the REF**1111 at (68.9, 99.7)
- removed the REF**1121 at (69.5, 99.7)
- removed the REF**1131 at (70.1, 99.7)
- removed the REF**1141 at (70.7, 99.7)
- removed the REF**1151 at (71.3, 99.7)
- removed the REF**1161 at (71.9, 99.7)
- removed TP40: TEST_POINT, 2kwMotorController:TEST_PAD_1.27mm
- added GNDISO: GND_POINT, Pin_Headers:Pin_Header_Straight_1x01, F.Cu at (71.0, 99.0)
- added GNDISO: GND_POINT, Pin_Headers:Pin_Header_Straight_1x01, F.Cu at (37.0, 22.0)
- added REF**: VIA-0.6mm, 2kwMotorController:VIA-0.6mm, F.Cu at (193.2, 84.2)
- added REF**: VIA-0.6mm, 2kwMotorController:VIA-0.6mm, F.Cu at (192.8, 84.2)
- added REF**: VIA-0.6mm, 2kwMotorController:VIA-0.6mm, F.Cu at (190.2, 84.2)
- added REF**: VIA-0.6mm, 2kwMotorController:VIA-0.6mm, F.Cu at (192.2, 84.2)
- added REF**: VIA-0.6mm, 2kwMotorController:VIA-0.6mm, F.Cu at (191.8, 84.2)
- added REF** (x2): VIA-0.6mm, 2kwMotorController:VIA-0.6mm, F.Cu at (191.2, 84.2)
- added REF** (x2): VIA-0.6mm, 2kwMotorController:VIA-0.6mm, F.Cu at (190.8, 84.2)
- C34, C40, C6, R10, R9: moved to B.Cu
- moved GNDISO 106.1 mm to (139.0, 22.0)
- moved R33 95.2 mm to (164.4, 69.5)
- moved GND 64.6 mm to (194.0, 32.5)
- moved GND2 63.7 mm to (179.0, 106.0)
- moved C12 52.0 mm to (164.8, 89.9), turned to 0 degrees
- moved SW2 52.0 mm to (164.8, 76.0), turned to 270 degrees
- moved C10 51.4 mm to (168.5, 89.9), turned to 180 degrees
- moved JP1 47.5 mm to (171.0, 82.0), turned to 90 degrees
- moved TP12 44.0 mm to (176.7, 28.0), turned to 270 degrees
- moved TP19 43.5 mm to (180.2, 67.5)
- moved C72 40.9 mm to (177.0, 43.0)
- moved R56 40.9 mm to (181.0, 43.0)
- moved REF**11 40.9 mm to (182.4, 43.9)
- moved REF**12 40.9 mm to (178.1, 44.5)
- moved REF**13 40.9 mm to (178.7, 44.5)
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- renumbered GND1 to GND, GND8 to GNDISO, GND9 to GNDISO
Connections:
- U13 pad 77: /mcu/CAN_ID_1 -> Net-(U13-Pad77)
- U13 pad 78: /mcu/CAN_ID_0 -> Net-(U13-Pad78)
Routing:
- net +BATT: track 29.6 -> 118.8 mm, vias 0 -> 1
- net +5V: track 6.53 -> 77.3 mm, vias 0 -> 3
- net +3V3: track 54.6 -> 109.6 mm, vias 18 -> 23
- net /mcu/PWM_FAN: track 2.36 -> 46.1 mm, vias 0 -> 2
- net /mcu/BRIDGE_TEMP: track 0.00 -> 41.2 mm, vias 0 -> 1
- net /mcu/MOTOR_TEMP: track 0.00 -> 34.5 mm
- net /mcu/LED_2: track 0.00 -> 33.7 mm
- net /mcu/LED_1: track 0.00 -> 32.0 mm
- net /mcu/LED_0: track 0.00 -> 30.2 mm
- net /mcu/DEBUG_0: track 17.7 -> 48.0 mm
- net /mcu/JTAG_RST_N: track 5.00 -> 35.0 mm, vias 0 -> 1
- net /mcu/QEI_IDX: track 0.00 -> 29.0 mm, vias 0 -> 4
- net /mcu/DEBUG_1: track 17.2 -> 46.1 mm
- net /mcu/DEBUG_2: track 16.8 -> 44.3 mm
- net /mcu/DEBUG_3: track 16.6 -> 42.6 mm
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- removed copper zone on F.Cu, net Net-(C52-Pad1)
Other:
- board size 170 x 97.8 mm -> 170 x 98.5 mm
- board text added: "+3V3"
- board text added: "GND IDX A 5V B"
- board text added: "GND PWR"
- board text removed: "FACTORY RESET"
- board text removed: "GND IDX A +5 B"
- board text removed: "GND ISO"
- board text removed: "ID0 ID1"
- board text removed: "UART"

Commit message: minor hw changes to submit PCB Rev 1
Parts:
- REF** (x6): footprint 2kwMotorController:M4-SCREW-HOLE -> 2kwMotorController:8MM_HOLE
- moved C57 6.40 mm to (74.5, 38.8), turned to 90 degrees
- moved U18 2.26 mm to (74.0, 44.5), turned to 90 degrees
- moved R2 2.15 mm to (141.3, 38.0), turned to 180 degrees
- moved C1 1.80 mm to (140.3, 34.8)
- moved C56 0.50 mm to (64.5, 51.0)
- moved C59 0.50 mm to (64.5, 48.5)
- moved C61 0.50 mm to (69.0, 51.5)
- moved C62 0.50 mm to (69.0, 49.8)
- moved REF**1111 0.50 mm to (70.7, 49.4)
- moved REF**1112 0.50 mm to (70.7, 49.9)
- moved REF**1113 0.50 mm to (70.7, 50.4)
- moved REF**1114 0.50 mm to (70.7, 50.9)
- moved REF**1115 0.50 mm to (70.7, 51.4)
- moved REF**1116 0.50 mm to (70.7, 51.9)
- moved REF**1111 0.50 mm to (64.1, 48.0)
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Routing:
- net Net-(R43-Pad1): track 22.9 -> 31.2 mm
- net Net-(R13-Pad1): track 19.5 -> 16.0 mm
- net /h-bridge/VBUS_ST_GD: track 73.7 -> 76.5 mm
- net +12V_ISO: track 275.8 -> 278.3 mm
- net Net-(C1-Pad1): track 7.59 -> 5.43 mm
- net /h-bridge/VBUS_EN_GD: track 74.0 -> 72.7 mm
- net Net-(C1-Pad2): track 23.5 -> 22.7 mm
- net Net-(R2-Pad1): track 2.41 -> 3.01 mm
- net GNDPWR: track 170.5 -> 170.0 mm

Commit message: Bugfixes and python terminal display
Parts:
- added GND1, GND8, GND9: GND_POINT, Pin_Headers:Pin_Header_Straight_1x01, F.Cu at (118.5, 126.1)
- added TP40: TEST_POINT, 2kwMotorController:TEST_PAD_1.27mm, F.Cu at (118.5, 126.1)
- C1: value 10p -> 56p
- C2: value 27n -> 1u
- C5: value 47n -> 2.2u
Changed lines of the file:
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@@
 (kicad_pcb (version 4) (host pcbnew 4.0.5+dfsg1-4)
   (general
-    (links 738)
-    (no_connects 5)
-    (area 25.9726 15.3226 209.295258 116.6274)
+    (links 742)
+    (no_connects 8)
+    (area 25.9726 15.3226 209.295258 128.601401)
     (thickness 1.6)
     (drawings 50)
     (tracks 1659)
     (zones 0)
-    (modules 415)
+    (modules 419)
     (nets 205)
   )
@@
     (33 F.Adhes user hide)
     (34 B.Paste user)
-    (35 F.Paste user)
+    (35 F.Paste user hide)
     (36 B.SilkS user)
     (37 F.SilkS user)
@@
   )
   (setup
-    (last_trace_width 0.508)
+    (last_trace_width 0.25)
     (user_trace_width 0.1524)
     (user_trace_width 0.254)
@@
       (effects (font (size 1 1) (thickness 0.15)))
     )
-    (fp_text value 10p (at 0 1.9 90) (layer F.Fab)
+    (fp_text value 56p (at 0 1.9 90) (layer F.Fab)
       (effects (font (size 1 1) (thickness 0.15)))
     )
@@
       (effects (font (size 1 1) (thickness 0.15)))
     )
-    (fp_text value 27n (at 0 1.9 180) (layer F.Fab)
+    (fp_text value 1u (at 0 1.9 180) (layer F.Fab)
       (effects (font (size 1 1) (thickness 0.15)))
     )
@@
       (effects (font (size 1 1) (thickness 0.15)))
     )
-    (fp_text value 47n (at 0 1.9 90) (layer F.Fab)
+    (fp_text value 2.2u (at 0 1.9 90) (layer F.Fab)
       (effects (font (size 1 1) (thickness 0.15)))
     )
@@
     (tags "capacitor 0603")
     (attr smd)
-    (fp_text reference C57 (at -3 0.25 270) (layer F.SilkS)
+    (fp_text reference C57 (at 0.95 3.4 360) (layer F.SilkS)
       (effects (font (size 1 1) (thickness 0.15)))
     )
@@
     (tags "resistor 0603")
     (attr smd)
-    (fp_text reference R38 (at 5.5 -0.25 450) (layer F.SilkS)
+    (fp_text reference R38 (at -2.9 0 180) (layer F.SilkS)
       (effects (font (size 1 1) (thickness 0.15)))
     )
@@
     (tags "capacitor 0603")
     (attr smd)
-    (fp_text reference C76 (at -6 0.25 360) (layer F.SilkS)
+    (fp_text reference C76 (at 2.25 0 450) (layer F.SilkS)
       (effects (font (size 1 1) (thickness 0.15)))
     )
@@
       (net 186 /h-bridge/VBUS_BRK_GATE))
   )
+  (module Pin_Headers:Pin_Header_Straight_1x01 (layer F.Cu)
+    (at 118.5 126.050001)
+    (descr "Through hole pin header")
+    (tags "pin header")
+    (fp_text reference GND1 (at 0 -5.1) (layer F.SilkS)
+      (effects (font (size 1 1) (thickness 0.15)))
+    )
+    (fp_text value GND_POINT (at 0 -3.1) (layer F.Fab)
+      (effects (font (size 1 1) (thickness 0.15)))
+    )
+    (fp_line (start 1.55 -1.55) (end 1.55 0) (layer F.SilkS) (width 0.15))
+    (fp_line (start -1.75 -1.75) (end -1.75 1.75) (layer F.CrtYd) (width 0.05))
+    (fp_line (start 1.75 -1.75) (end 1.75 1.75) (layer F.CrtYd) (width 0.05))
+    (fp_line (start -1.75 -1.75) (end 1.75 -1.75) (layer F.CrtYd) (width 0.05))
+    (fp_line (start -1.75 1.75) (end 1.75 1.75) (layer F.CrtYd) (width 0.05))
+    (fp_line (start -1.55 0) (end -1.55 -1.55) (layer F.SilkS) (width 0.15))
+    (fp_line (start -1.55 -1.55) (end 1.55 -1.55) (layer F.SilkS) (width 0.15))
+    (fp_line (start -1.27 1.27) (end 1.27 1.27) (layer F.SilkS) (width 0.15))
+    (pad 1 thru_hole rect (at 0 0) (size 2.2352 2.2352) (drill 1.016) (layers *.Cu *.Mask)
+      (net 3 GND))
+    (model Pin_Headers.3dshapes/Pin_Header_Straight_1x01.wrl
+      (at (xyz 0 0 0))
+      (scale (xyz 1 1 1))
+      (rotate (xyz 0 0 90))
+    )
+  )
+  (module Pin_Headers:Pin_Header_Straight_1x01 (layer F.Cu)
+    (at 118.5 126.050001)
+    (descr "Through hole pin header")
+    (tags "pin header")
+    (fp_text reference GND8 (at 0 -5.1) (layer F.SilkS)
+      (effects (font (size 1 1) (thickness 0.15)))
+    )
+    (fp_text value GND_POINT (at 0 -3.1) (layer F.Fab)
+      (effects (font (size 1 1) (thickness 0.15)))
+    )
+    (fp_line (start 1.55 -1.55) (end 1.55 0) (layer F.SilkS) (width 0.15))
+    (fp_line (start -1.75 -1.75) (end -1.75 1.75) (layer F.CrtYd) (width 0.05))
+    (fp_line (start 1.75 -1.75) (end 1.75 1.75) (layer F.CrtYd) (width 0.05))
+    (fp_line (start -1.75 -1.75) (end 1.75 -1.75) (layer F.CrtYd) (width 0.05))
+    (fp_line (start -1.75 1.75) (end 1.75 1.75) (layer F.CrtYd) (width 0.05))
+    (fp_line (start -1.55 0) (end -1.55 -1.55) (layer F.SilkS) (width 0.15))
+    (fp_line (start -1.55 -1.55) (end 1.55 -1.55) (layer F.SilkS) (width 0.15))
+    (fp_line (start -1.27 1.27) (end 1.27 1.27) (layer F.SilkS) (width 0.15))
+    (pad 1 thru_hole rect (at 0 0) (size 2.2352 2.2352) (drill 1.016) (layers *.Cu *.Mask)
+      (net 10 GNDPWR))
+    (model Pin_Headers.3dshapes/Pin_Header_Straight_1x01.wrl
+      (at (xyz 0 0 0))
+      (scale (xyz 1 1 1))
+      (rotate (xyz 0 0 90))
+    )
+  )
+  (module Pin_Headers:Pin_Header_Straight_1x01 (layer F.Cu)
+    (at 118.5 126.050001)
+    (descr "Through hole pin header")
+    (tags "pin header")
+    (fp_text reference GND9 (at 0 -5.1) (layer F.SilkS)
+      (effects (font (size 1 1) (thickness 0.15)))
+    )
+    (fp_text value GND_POINT (at 0 -3.1) (layer F.Fab)
+      (effects (font (size 1 1) (thickness 0.15)))
+    )
+    (fp_line (start 1.55 -1.55) (end 1.55 0) (layer F.SilkS) (width 0.15))
+    (fp_line (start -1.75 -1.75) (end -1.75 1.75) (layer F.CrtYd) (width 0.05))
+    (fp_line (start 1.75 -1.75) (end 1.75 1.75) (layer F.CrtYd) (width 0.05))
+    (fp_line (start -1.75 -1.75) (end 1.75 -1.75) (layer F.CrtYd) (width 0.05))
+    (fp_line (start -1.75 1.75) (end 1.75 1.75) (layer F.CrtYd) (width 0.05))
+    (fp_line (start -1.55 0) (end -1.55 -1.55) (layer F.SilkS) (width 0.15))
+    (fp_line (start -1.55 -1.55) (end 1.55 -1.55) (layer F.SilkS) (width 0.15))
+    (fp_line (start -1.27 1.27) (end 1.27 1.27) (layer F.SilkS) (width 0.15))
+    (pad 1 thru_hole rect (at 0 0) (size 2.2352 2.2352) (drill 1.016) (layers *.Cu *.Mask)
+      (net 10 GNDPWR))
+    (model Pin_Headers.3dshapes/Pin_Header_Straight_1x01.wrl
+      (at (xyz 0 0 0))
+      (scale (xyz 1 1 1))
+      (rotate (xyz 0 0 90))
+    )
+  )
+  (module 2kwMotorController:TEST_PAD_1.27mm (layer F.Cu)
+    (at 118.5 126.050001)
+    (fp_text reference TP40 (at 0 1.524) (layer F.SilkS)
+      (effects (font (size 1 1) (thickness 0.15)))
+    )
+    (fp_text value TEST_POINT (at 0 -1.524) (layer F.Fab) hide
+      (effects (font (size 1 1) (thickness 0.15)))
+    )
+    (pad 1 thru_hole circle (at 0 0) (size 1.524 1.524) (drill 0.762) (layers *.Cu *.Mask F.SilkS)
+      (net 15 +12V_ISO))
+  )
   (gr_text +3V3 (at 181.5 27) (layer F.SilkS)
