File: hardware/_saved_power.sch (KiCad schematic (older format))
At the start: 65 parts, among them P1 CONN_01X02_CBAT, P2 CONN_01X02_FAN, Q1 DMG4712SSS, Q2 DMG4712SSS, U10 MCP1501T-30E, U11 PDM1-S, U12 MIC5225-5.0, U7 MIC5225-5.0, U8 LT3471, U9 R-78E3.3-0.5

Commit message: more layout progress
Changed lines of the file:
@@
 	7500 1550 7500 1650
 Wire Wire Line
-	6300 1150 6300 1300
+	6300 1300 6300 1150
 Connection ~ 6300 1150
 Wire Wire Line
