File: hardware/_saved_power.sch (KiCad schematic (older format))
At the start: 67 parts, among them P1 CONN_01X02_CBAT, P2 CONN_01X02_FAN, Q1 DMG4712SSS, Q2 DMG4712SSS, U10 MCP1501T-30E, U11 PDM1-S, U12 MIC5225-5.0, U7 MIC5225-5.0, U8 LT3471, U9 R-78E3.3-0.5

Commit message: layout cleanup, add buffer for fan drive
Parts:
- C82: renamed from C?; footprint (none) -> Capacitors_SMD:C_0603
- gave numbers to parts that had none: 1
