File: hardware/_saved_h-bridge.sch (KiCad schematic (older format))
At the start: 83 parts, among them M1 MOUNTING_HOLE, M2 MOUNTING_HOLE, M3 MOUNTING_HOLE, M4 MOUNTING_HOLE, M5 MOUNTING_HOLE, M6 MOUNTING_HOLE, P10 CONN_01_BRK, P11 CONN_01_M+, P12 CONN_01_M-, P8 CONN_01_V+, P9 CONN_01_V-, Q10 PSMN021-100, Q3 IRFP4468, Q4 PSMN021-100, Q5 IRFP4468, Q6 IRFP4468, Q7 IRFP4468, Q8 IRFP4468, Q9 IRFP4468, U16 Si8045AA, U17 MIC4127, U18 MIC4127, U19 UCC27211, U20 Si8045AA, U6 UCC27211

Commit message: tweaks, testpoints, decluttering
Parts:
- gave numbers to parts that had none: 4
Changed lines of the file:
@@
 $EndComp
 $Comp
-L GNDPWR #PWR?
+L GNDPWR #PWR0126
 U 1 1 59CAF326
 P 5900 6250
-F 0 "#PWR?" H 5900 6050 50  0001 C CNN
+F 0 "#PWR0126" H 5900 6050 50  0001 C CNN
 F 1 "GNDPWR" H 5900 6120 50  0000 C CNN
 F 2 "" H 5900 6200 50  0000 C CNN
@@
 $EndComp
 $Comp
-L GND_POINT GND?
+L GND_POINT GND8
 U 1 1 59CAF458
 P 5900 6100
-F 0 "GND?" H 5900 6300 60  0001 C CNN
+F 0 "GND8" H 5900 6300 60  0001 C CNN
 F 1 "GND_POINT" H 5925 6375 60  0001 C CNN
 F 2 "2kwMotorController:TEST_PAD_1.27mm" H 5900 6100 60  0001 C CNN
@@
 	5900 6100 5900 6250
 $Comp
-L GND_POINT GND?
+L GND_POINT GND9
 U 1 1 59CB0A30
 P 6100 6100
-F 0 "GND?" H 6100 6300 60  0001 C CNN
+F 0 "GND9" H 6100 6300 60  0001 C CNN
 F 1 "GND_POINT" H 6125 6375 60  0001 C CNN
 F 2 "2kwMotorController:TEST_PAD_1.27mm" H 6100 6100 60  0001 C CNN
@@
 $EndComp
 $Comp
-L GND_POINT GND?
+L GND_POINT GND10
 U 1 1 59CB0B13
 P 6300 6100
-F 0 "GND?" H 6300 6300 60  0001 C CNN
+F 0 "GND10" H 6300 6300 60  0001 C CNN
 F 1 "GND_POINT" H 6325 6375 60  0001 C CNN
 F 2 "2kwMotorController:TEST_PAD_1.27mm" H 6300 6100 60  0001 C CNN
@@
 $EndComp
 $Comp
-L GND_POINT GND?
+L GND_POINT GND11
 U 1 1 59CB0BF6
 P 6500 6100
-F 0 "GND?" H 6500 6300 60  0001 C CNN
+F 0 "GND11" H 6500 6300 60  0001 C CNN
 F 1 "GND_POINT" H 6525 6375 60  0001 C CNN
 F 2 "2kwMotorController:TEST_PAD_1.27mm" H 6500 6100 60  0001 C CNN
