File: hardware/2kwMotorController.sch (KiCad schematic (older format))
At the start: 0 parts

Commit message: Rev 1 layout finished
Other:
- note removed: "h-bridge decoupling\nCAN connection\nconnectors\nVDDA filter"
Changed lines of the file:
@@
 Wire Wire Line
 	2700 2800 3350 2800
-Text Notes 8400 5450 0    157  ~ 31
-h-bridge decoupling\nCAN connection\nconnectors\nVDDA filter
 Wire Wire Line
 	4950 2900 5200 2900
